File: pcb/tweezer.sch (EAGLE design)
At the start: 33 parts, among them IC1 AD7995, IC2 TS507CLT, IC3 TS507CLT, IC5 ESDA6V1SC5, IC6 AT24CS04-SOT23

Commit message: fixing op amp (iron,tweezer)
Changed lines of the file:
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@@
 <?xml version="1.0" encoding="utf-8"?>
 <!DOCTYPE eagle SYSTEM "eagle.dtd">
-<eagle version="9.0.0">
+<eagle version="9.0.1">
 <drawing>
 <settings>
@@
 <part name="GND1" library="supply1" library_urn="urn:adsk.eagle:library:371" deviceset="GND" device=""/>
 <part name="R1" library="rcl" library_urn="urn:adsk.eagle:library:334" deviceset="R-EU_" device="R0805" package3d_urn="urn:adsk.eagle:package:23553/2"/>
-<part name="R2" library="solderpi" library_urn="urn:adsk.eagle:library:1437534" deviceset="NTC-0805" device="" package3d_urn="urn:adsk.eagle:package:1581953/3" value="330k @25°C, 1%, ß=3930"/>
+<part name="R2" library="solderpi" library_urn="urn:adsk.eagle:library:1437534" deviceset="NTC-0805" device="" package3d_urn="urn:adsk.eagle:package:1581953/4" value="330k @25°C, 1%, ß=3930"/>
 <part name="P+1" library="supply1" library_urn="urn:adsk.eagle:library:371" deviceset="+5V" device=""/>
 <part name="GND3" library="supply1" library_urn="urn:adsk.eagle:library:371" deviceset="GND" device=""/>
@@
 <part name="R10" library="rcl" library_urn="urn:adsk.eagle:library:334" deviceset="R-EU_" device="R0805" package3d_urn="urn:adsk.eagle:package:23553/2" value="2k"/>
 <part name="GND6" library="supply1" library_urn="urn:adsk.eagle:library:371" deviceset="GND" device=""/>
-<part name="IC2" library="solderpi" library_urn="urn:adsk.eagle:library:1437534" deviceset="TS507CLT" device="" package3d_urn="urn:adsk.eagle:package:1437676/5"/>
+<part name="IC2" library="solderpi" library_urn="urn:adsk.eagle:library:1437534" deviceset="TS507CLT" device="" package3d_urn="urn:adsk.eagle:package:1437676/7"/>
 <part name="GND7" library="supply1" library_urn="urn:adsk.eagle:library:371" deviceset="GND" device=""/>
 <part name="GND8" library="supply1" library_urn="urn:adsk.eagle:library:371" deviceset="GND" device=""/>
@@
 <part name="R14" library="rcl" library_urn="urn:adsk.eagle:library:334" deviceset="R-EU_" device="R0805" package3d_urn="urn:adsk.eagle:package:23553/2" value="2k"/>
 <part name="GND10" library="supply1" library_urn="urn:adsk.eagle:library:371" deviceset="GND" device=""/>
-<part name="IC3" library="solderpi" library_urn="urn:adsk.eagle:library:1437534" deviceset="TS507CLT" device="" package3d_urn="urn:adsk.eagle:package:1437676/5"/>
+<part name="IC3" library="solderpi" library_urn="urn:adsk.eagle:library:1437534" deviceset="TS507CLT" device="" package3d_urn="urn:adsk.eagle:package:1437676/7"/>
 <part name="GND11" library="supply1" library_urn="urn:adsk.eagle:library:371" deviceset="GND" device=""/>
 <part name="GND12" library="supply1" library_urn="urn:adsk.eagle:library:371" deviceset="GND" device=""/>
@@
 <part name="P+4" library="supply1" library_urn="urn:adsk.eagle:library:371" deviceset="+5V" device=""/>
 <part name="ß" library="solderpi" library_urn="urn:adsk.eagle:library:1437534" deviceset="WIREPAD" device="" package3d_urn="urn:adsk.eagle:package:1593774/7"/>
-<part name="IC5" library="solderpi" library_urn="urn:adsk.eagle:library:1437534" deviceset="ESDA6V1SC5" device="" package3d_urn="urn:adsk.eagle:package:1437676/5"/>
+<part name="IC5" library="solderpi" library_urn="urn:adsk.eagle:library:1437534" deviceset="ESDA6V1SC5" device="" package3d_urn="urn:adsk.eagle:package:1437676/7"/>
 <part name="GND13" library="supply1" library_urn="urn:adsk.eagle:library:371" deviceset="GND" device=""/>
 <part name="P+11" library="supply1" library_urn="urn:adsk.eagle:library:371" deviceset="+5V" device=""/>
-<part name="IC6" library="solderpi" library_urn="urn:adsk.eagle:library:1437534" deviceset="AT24CS04-SOT23" device="" package3d_urn="urn:adsk.eagle:package:1437676/5"/>
+<part name="IC6" library="solderpi" library_urn="urn:adsk.eagle:library:1437534" deviceset="AT24CS04-SOT23" device="" package3d_urn="urn:adsk.eagle:package:1437676/7"/>
 </parts>
 <sheets>
