File: pcb/controller.brd (EAGLE design)
At the start: 100 x 66.4 mm, 165 parts, among them IC1 LTC4357, IC10 ST2378E, IC11 5k, IC12 LT1803, IC13 INA196, IC14 INA196, IC15 INA196, IC16 INA196, IC17 INA196, IC18 INA196, IC2 LM1084, IC3 LMR62014, IC4 LM74670, IC5 LM74670, IC6 LM74670, IC7 LM74670, IC8 ATSAMC21J, IC9 PCA9533, Q1 24MHz, Q2 32768kHz, T1 FDS6670A, T10 NVR4003NT3G, T11 NVR4003NT3G, T12 IRF9392PBF, T13 IRF9392PBF, T14 NVR4003NT3G, T15 IRF9392PBF, T16 NVR4003NT3G, T17 IRF9392PBF, T18 BSS7728NH6327XTSA1, T19 BSS84PH6433XTMA1, T2 PSMN1R0, T20 BSS84PH6433XTMA1, T21 BSS84PH6433XTMA1, T3 PSMN1R0, T4 PSMN1R0, T5 PSMN1R0, T6 NVR4003NT3G, T7 NVR4003NT3G, T8 IRF9392PBF, T9 IRF9392PBF, X1 ULTRAFIT-20, X10 IGRID-14, X11 MICRO-CLASP-6, X2 NANOFIT-7, X3 NANOFIT-7, X4 NANOFIT-7, X5 JTAG-EDGE-CON, X6 B3S-1000, X7 IGRID-10, X9 MICRO-LATCH-4

Commit message: updated Schematic from lib
Routing:
- net GND: track 862.6 -> 861.4 mm
Changed lines of the file:
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@@
 <?xml version="1.0" encoding="utf-8"?>
 <!DOCTYPE eagle SYSTEM "eagle.dtd">
-<eagle version="9.0.1">
+<eagle version="9.2.2">
 <drawing>
 <settings>
@@
 <setting verticaltext="up"/>
 </settings>
-<grid distance="0.4" unitdist="mm" unit="mm" style="lines" multiple="1" display="no" altdistance="0.05" altunitdist="mm" altunit="mm"/>
+<grid distance="1" unitdist="mm" unit="mm" style="lines" multiple="1" display="no" altdistance="0.05" altunitdist="mm" altunit="mm"/>
 <layers>
-<layer number="1" name="Top" color="4" fill="1" visible="yes" active="yes"/>
+<layer number="1" name="Top" color="4" fill="1" visible="no" active="yes"/>
 <layer number="2" name="Route2" color="1" fill="3" visible="no" active="no"/>
 <layer number="3" name="Route3" color="4" fill="3" visible="no" active="no"/>
@@
 <layer number="19" name="Unrouted" color="6" fill="1" visible="yes" active="yes"/>
 <layer number="20" name="Dimension" color="24" fill="1" visible="yes" active="yes"/>
-<layer number="21" name="tPlace" color="7" fill="1" visible="yes" active="yes"/>
+<layer number="21" name="tPlace" color="7" fill="1" visible="no" active="yes"/>
 <layer number="22" name="bPlace" color="7" fill="1" visible="yes" active="yes"/>
-<layer number="23" name="tOrigins" color="15" fill="1" visible="yes" active="yes"/>
+<layer number="23" name="tOrigins" color="15" fill="1" visible="no" active="yes"/>
 <layer number="24" name="bOrigins" color="15" fill="1" visible="yes" active="yes"/>
-<layer number="25" name="tNames" color="7" fill="1" visible="yes" active="yes"/>
-<layer number="26" name="bNames" color="7" fill="1" visible="yes" active="yes"/>
+<layer number="25" name="tNames" color="7" fill="1" visible="no" active="yes"/>
+<layer number="26" name="bNames" color="7" fill="1" visible="no" active="yes"/>
 <layer number="27" name="tValues" color="7" fill="1" visible="no" active="yes"/>
 <layer number="28" name="bValues" color="7" fill="1" visible="no" active="yes"/>
@@
 <layer number="37" name="tTest" color="7" fill="1" visible="no" active="yes"/>
 <layer number="38" name="bTest" color="7" fill="1" visible="no" active="yes"/>
-<layer number="39" name="tKeepout" color="4" fill="11" visible="yes" active="yes"/>
+<layer number="39" name="tKeepout" color="4" fill="11" visible="no" active="yes"/>
 <layer number="40" name="bKeepout" color="1" fill="11" visible="yes" active="yes"/>
-<layer number="41" name="tRestrict" color="4" fill="10" visible="yes" active="yes"/>
-<layer number="42" name="bRestrict" color="1" fill="10" visible="yes" active="yes"/>
-<layer number="43" name="vRestrict" color="2" fill="10" visible="yes" active="yes"/>
+<layer number="41" name="tRestrict" color="4" fill="10" visible="no" active="yes"/>
+<layer number="42" name="bRestrict" color="1" fill="10" visible="no" active="yes"/>
+<layer number="43" name="vRestrict" color="2" fill="10" visible="no" active="yes"/>
 <layer number="44" name="Drills" color="7" fill="1" visible="no" active="yes"/>
 <layer number="45" name="Holes" color="7" fill="1" visible="yes" active="yes"/>
@@
 <layer number="48" name="Document" color="7" fill="1" visible="no" active="yes"/>
 <layer number="49" name="Reference" color="7" fill="1" visible="no" active="yes"/>
-<layer number="51" name="tDocu" color="7" fill="1" visible="yes" active="yes"/>
-<layer number="52" name="bDocu" color="7" fill="1" visible="yes" active="yes"/>
+<layer number="51" name="tDocu" color="7" fill="1" visible="no" active="yes"/>
+<layer number="52" name="bDocu" color="7" fill="1" visible="no" active="yes"/>
 <layer number="88" name="SimResults" color="9" fill="1" visible="no" active="no"/>
 <layer number="89" name="SimProbes" color="9" fill="1" visible="no" active="no"/>
@@
 <param name="checkStop" value="0"/>
 <param name="checkValues" value="1"/>
+<param name="checkNames" value="1"/>
+<param name="checkWireStubs" value="1"/>
+<param name="checkPolygonWidth" value="0"/>
 <param name="useDiameter" value="13"/>
 <param name="maxErrors" value="50"/>
@@
 <wire x1="50.25" y1="48" x2="45.45" y2="48" width="0.2" layer="16"/>
 <wire x1="50.25" y1="50.15" x2="50.25" y2="48" width="0.2" layer="16"/>
-<wire x1="28.6476" y1="43.8476" x2="28.6476" y2="36.8" width="0.2" layer="16"/>
+<wire x1="28.6476" y1="41.8476" x2="28.6476" y2="36.8" width="0.2" layer="16"/>
 <via x="31.6" y="48.4" extent="1-16" drill="0.3"/>
 <wire x1="36.1" y1="50.4" x2="34.8" y2="50.4" width="0.2" layer="16"/>
@@
 <wire x1="41.1" y1="33.1" x2="41.1" y2="33.1226" width="0.2" layer="16"/>
 <wire x1="41.1" y1="33.1226" x2="41.35" y2="33.3726" width="0.2" layer="16"/>
-<wire x1="29.55" y1="44.75" x2="28.6476" y2="43.8476" width="0.2" layer="16"/>
+<wire x1="31.55" y1="44.75" x2="28.6476" y2="41.8476" width="0.2" layer="16"/>
 <wire x1="41.05" y1="44.75" x2="32.4" y2="44.75" width="0.2" layer="16"/>
-<wire x1="32.4" y1="44.75" x2="29.55" y2="44.75" width="0.2" layer="16"/>
+<wire x1="32.4" y1="44.75" x2="31.55" y2="44.75" width="0.2" layer="16"/>
 <wire x1="32.4" y1="47.6" x2="32.4" y2="44.75" width="0.2" layer="16"/>
 <via x="33.83335" y="49.03335" extent="1-16" drill="0.3"/>
@@
 </signal>
 </signals>
+<mfgpreviewcolors>
+<mfgpreviewcolor name="soldermaskcolor" color="0xC8008000"/>
+<mfgpreviewcolor name="silkscreencolor" color="0xFFFEFEFE"/>
+<mfgpreviewcolor name="backgroundcolor" color="0xFF282828"/>
+<mfgpreviewcolor name="coppercolor" color="0xFFFFBF00"/>
+<mfgpreviewcolor name="substratecolor" color="0xFF786E46"/>
+</mfgpreviewcolors>
 <errors>
 </errors>
