File: pcb/controller.brd (EAGLE design)
At the start: 120 x 100 mm, 88 parts, among them IC1 STM32L496X, IC2 TPS62173, IC3 TPS62162, IC4 INA196, IC5 INA196, IC6 INA196, IC7 INA196, Q1 24Mhz, SW1 EC12E_SW, SW2 EC12E_SW, T1 NVR4003NT3G, T2 NVR4003NT3G, T3 IRF7416, T4 IRF7416, T5 NVR4003NT3G, T6 NVR4003NT3G, T7 IRF7416, T8 IRF7416, X1 NEWHAVEN_OLED_256X64, X2 ULTRAFIT-290, X3 PINHD-1X2, X4 NANOFIT-7, X5 PINHD-1X2, X6 NANOFIT-7

Commit message: shottky diode added to iron/tweezer
Parts:
- moved C18 234.4 mm to (110.0, 11.0), flipped to the bottom, turned to 180 degrees
- moved R42 224.2 mm to (110.0, 13.0), flipped to the bottom
- moved C17 216.0 mm to (117.3, 7.90)
- moved R37 206.7 mm to (100.0, 11.0)
- moved L2 204.9 mm to (73.0, 13.3), turned to 270 degrees
- moved R5 204.2 mm to (70.3, 9.40)
- moved IC2 199.8 mm to (68.0, 22.0)
- moved L1 196.8 mm to (73.0, 23.4), turned to 270 degrees
- moved R40 195.1 mm to (115.0, 4.00)
- moved R4 194.3 mm to (70.8, 19.4)
- moved C16 193.5 mm to (99.0, 8.00)
- moved R41 188.9 mm to (109.0, 18.0), flipped to the bottom
- moved R33 180.2 mm to (76.5, 68.1), turned to 90 degrees
- moved R39 179.6 mm to (109.0, 3.00)
- moved R35 178.8 mm to (103.0, 5.00)
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Routing:
- net +3V3: track 0.00 -> 11.1 mm, vias 0 -> 2
- net GND: track 0.00 -> 8.89 mm, vias 0 -> 5
- net +5V: track 0.00 -> 7.65 mm
- net 3V3_PG: track 0.00 -> 5.59 mm, vias 0 -> 2
- net 3V3_SW: track 0.00 -> 4.12 mm
- net 5V_SW: track 0.00 -> 4.05 mm
- net +12V: track 0.00 -> 3.38 mm
Other:
- outline, holes or cut-outs redrawn

Commit message: iron tweezer updated
Parts:
- added C19, C20: 12pF, rcl:C0603
- added X7: PINHD-1X4, solderpi:1X04
- added X8: PINHD-1X3, solderpi:1X03
- added X9: PINHD-1X6, solderpi:1X06
- C1, C2, C3, C4, C5, C6, C7: device rcl:C0603 -> rcl:C0402
- X3: value PINHD-1X2 -> PINHD-1X3; device solderpi:1X02 -> solderpi:1X03
- X5: value PINHD-1X2 -> PINHD-1X4; device solderpi:1X02 -> solderpi:1X04
- moved R1 192.4 mm to (89.5, 52.2), turned to 270 degrees
- moved R27 186.5 mm to (77.1, 63.0), turned to 270 degrees
- moved R2 171.0 mm to (56.4, 21.3), flipped to the bottom, turned to 270 degrees
- moved T8 166.6 mm to (68.4, 62.0), flipped to the bottom, turned to 90 degrees
- moved X1 162.4 mm to (50.0, 45.0)
- moved R32 161.9 mm to (78.0, 66.0), flipped to the bottom
- moved Q1 161.8 mm to (51.5, 47.6), turned to 180 degrees
- moved R3 160.8 mm to (60.8, 41.0), turned to 270 degrees
- moved T7 159.4 mm to (71.1, 62.0), turned to 90 degrees
- moved C4 158.0 mm to (48.0, 44.2), flipped to the bottom
- moved R31 154.2 mm to (74.9, 66.0), flipped to the bottom
- moved C7 152.1 mm to (48.0, 43.1), flipped to the bottom
- moved C3 148.9 mm to (53.5, 31.9), flipped to the bottom
- moved X5 148.6 mm to (87.3, 21.5), flipped to the bottom
- moved C5 146.7 mm to (44.3, 34.0), flipped to the bottom, turned to 90 degrees
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Connections:
- net N$37 renamed BOOT0
- net +3V3: now also C6.1, R40.2; no longer C7.1, R23.2
- net +3V3_ANA: now also C7.1; no longer C6.1
- net AGND: now also C7.2; no longer C6.2
- net CHA0_SCL: now also IC1.29, X8.1; no longer IC1.58, X3.1
- net CHA0_SDA: now also IC1.30, X8.2; no longer IC1.59, X3.2
- net CHA0_TIP0_CUR: now also IC1.17; no longer IC1.9
- net CHA0_TIP0_PWM: now also IC1.42; no longer IC1.44
- net CHA0_TIP0_VOL: now also IC1.16; no longer IC1.8
- net CHA0_TIP1_CUR: now also IC1.14; no longer IC1.11
- net CHA0_TIP1_PWM: now also IC1.41; no longer IC1.43
- net CHA0_TIP1_VOL: now also IC1.15; no longer IC1.10
- net CHA1_SCL: now also IC1.58, X3.1; no longer IC1.29, X5.1
- net CHA1_SDA: now also IC1.59, X3.2; no longer IC1.30, X5.2
- net CHA1_TIP0_CUR: now also IC1.11; no longer IC1.15
- net CHA1_TIP0_PWM: now also IC1.44; no longer IC1.42
- net CHA1_TIP0_VOL: now also IC1.10; no longer IC1.14
- net CHA1_TIP1_CUR: now also IC1.9; no longer IC1.17
- net CHA1_TIP1_PWM: now also IC1.43; no longer IC1.41
- net CHA1_TIP1_VOL: now also IC1.8; no longer IC1.16
- net ENC0_A: now also IC1.23, X7.1; no longer IC1.52
- net ENC0_B: now also IC1.21, R22.1, X7.3; no longer IC1.50, R22.2
- net ENC0_B_UNFIL: now also R22.2; no longer R22.1
- net ENC0_SW: now also IC1.22, X7.2; no longer IC1.51
- net ENC0_SW_R: now also R41.1; no longer R23.1
- net ENC1_A: now also IC1.52, R23.1, X5.2; no longer IC1.21, R35.1
- net ENC1_A_UNFIL: now also R23.2; no longer R35.2
- net ENC1_B: now also IC1.50, R35.2, X5.4; no longer IC1.23, R40.2
- net ENC1_B_UNFIL: now also R35.1; no longer R40.1
- net ENC1_SW: now also IC1.51, X5.3; no longer IC1.22
- net ENC1_SW_R: now also R40.1; no longer R41.1
- net GND: now also C19.2, C20.2, C6.2, X3.3, X5.1, X7.4, X8.3, X9.6; no longer C7.2
- net OLED_!CS: now also X9.5
- net OLED_!RESET: now also X9.4
- net OLED_D/C: now also X9.1
- net OLED_SDCLK: now also X9.2
- net OLED_SDIN: now also X9.3
- net OSC_IN: now also C20.1
- net OSC_OUT: now also C19.1
Routing:
- net GND: track 8.89 -> 451.6 mm, vias 5 -> 13
- net +3V3: track 11.1 -> 204.3 mm, vias 2 -> 12
- net +12V: track 3.38 -> 147.4 mm, vias 0 -> 4
- net CHA1_SCL: track 0.00 -> 78.0 mm
- net CHA1_SDA: track 0.00 -> 72.5 mm
- net +5V: track 7.65 -> 72.7 mm, vias 0 -> 2
- net AGND: track 0.00 -> 61.5 mm, vias 0 -> 3
- net ENC0_SW: track 0.00 -> 60.6 mm, vias 0 -> 1
- net ENC0_B: track 0.00 -> 59.7 mm
- net ENC0_A: track 0.00 -> 58.1 mm
- net ENC1_A: track 0.00 -> 55.5 mm
- net ENC1_SW: track 0.00 -> 55.1 mm, vias 0 -> 1
- net ENC1_B: track 0.00 -> 54.0 mm
- net SWDIO: track 0.00 -> 49.3 mm, vias 0 -> 1
- net SWO: track 0.00 -> 49.0 mm
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Other:
- board size 120 x 100 mm -> 100 x 100 mm

Commit message: boms reworked
Parts:
- removed C11: 22µ, rcl:C0805
- removed C8: 10µ, rcl:C0805
- removed IC2: TPS62173, solderpi:WSON8
- removed L1: (no value), solderpi:VLF3012ST
- removed L3: 300R @ 100MHz, solderpi:L0603
- removed R4: 100k, rcl:R0603
- removed R6: 0, rcl:R2010
- moved C19 11.4 mm to (50.6, 39.1), flipped to the bottom, turned to 270 degrees
- moved C20 11.4 mm to (52.8, 39.1), flipped to the bottom, turned to 270 degrees
- moved C12 5.00 mm to (23.4, 42.4)
- moved C9 5.00 mm to (24.3, 46.1)
- moved IC3 5.00 mm to (25.7, 43.1)
- moved L2 5.00 mm to (24.4, 38.1)
- moved R5 5.00 mm to (28.4, 40.8)
- moved Q1 4.80 mm to (51.7, 42.9), flipped to the bottom, turned to 0 degrees
- moved C10 4.00 mm to (20.9, 62.5)
- moved IC4 4.00 mm to (47.3, 66.7)
- moved IC5 4.00 mm to (36.2, 66.7)
- moved IC6 4.00 mm to (64.2, 66.7)
- moved IC7 4.00 mm to (75.3, 66.7)
- moved R10 4.00 mm to (49.1, 59.0)
- moved R11 4.00 mm to (46.9, 62.0)
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Connections:
- removed net +3V3_ANA: C2.1, C4.1, C7.1, IC1.12, IC4.3, IC5.3, IC6.3, IC7.3, L3.1
- removed net +5V: C11.1, IC2.6, L1.1, R19.2, R21.2, R36.2, R38.2, R4.2, X4.3, X6.3
- removed net 5V_PG: IC2.8, R4.1
- removed net 5V_SW: IC2.7, L1.2
- removed net AGND: C2.2, C4.2, C7.2, IC1.13, IC4.2, IC5.2, IC6.2, IC7.2, R6.2
- net +12V: no longer C8.1, IC2.2, IC2.3
- net +3V3: now also C2.1, C4.1, C7.1, IC1.12, IC4.3, IC5.3, IC6.3, IC7.3, R19.2, R21.2, R36.2, R38.2, X4.3, X6.3; no longer L3.2
- net CHA1_TIP1_CUR: now also IC1.8; no longer IC1.9
- net CHA1_TIP1_VOL: now also IC1.9; no longer IC1.8
- net GND: now also C2.2, C4.2, C7.2, IC1.13, IC4.2, IC5.2, IC6.2, IC7.2; no longer C11.2, C8.2, IC2.1, IC2.4, IC2.5, IC2.GND, R6.1
Routing:
- net +3V3: track 204.3 -> 376.5 mm, vias 12 -> 19
- net GND: track 451.6 -> 600.2 mm, vias 13 -> 19
- net +5V: track 72.7 -> 0.00 mm, vias 2 -> 0
- net AGND: track 61.5 -> 0.00 mm, vias 3 -> 0
- net CHA1_TIP1_CUR: track 0.00 -> 51.1 mm, vias 0 -> 1
- net RESET: track 0.00 -> 46.9 mm, vias 0 -> 1
- net CHA1_TIP0_PWM: track 3.95 -> 50.1 mm, vias 0 -> 2
- net CHA1_TIP1_VOL: track 1.35 -> 46.4 mm, vias 0 -> 1
- net CHA0_TIP0_CUR: track 4.81 -> 49.7 mm, vias 0 -> 2
- net CHA0_SDA: track 10.2 -> 54.4 mm, vias 0 -> 3
- net CHA0_TIP0_VOL: track 3.26 -> 45.1 mm, vias 0 -> 2
- net CHA0_TIP0_PWM: track 3.90 -> 43.5 mm, vias 0 -> 4
- net CHA0_SCL: track 12.3 -> 50.7 mm, vias 1 -> 2
- net CHA0_TIP1_PWM: track 3.95 -> 41.8 mm, vias 0 -> 3
- net CHA1_TIP0_CUR: track 0.00 -> 32.8 mm, vias 0 -> 2
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- added copper zone on layer 1, net +12V
- added copper zone on layer 16, net +12V
- added copper zone on layer 1, net CHA0_TIP0_SEN
- added copper zone on layer 16, net CHA0_TIP1_SEN
- added copper zone on layer 1, net CHA1_TIP0
- added copper zone on layer 1, net CHA1_TIP0_SEN
- added copper zone on layer 16, net CHA1_TIP1
- added copper zone on layer 16, net CHA1_TIP1_SEN
- added copper zone on layer 1, net GND
- added copper zone on layer 16, net GND
Other:
- board size 100 x 100 mm -> 100 x 94 mm
- board text added: "!CS"
- board text added: "!RES"
- board text added: "D/C"
- board text added: "SDCLK"
- board text added: "SDIN"
