File: pcb/iron.sch (EAGLE design)
At the start: 22 parts, among them IC1 AT24CS04-SOT23, IC2 TS507CLT, IC3 AD7995, IC4 ESDA6V1SC5, X1 LUMBERG_KLB_4

Commit message: fixed vcc,vdd on opAmp
Connections:
- net +5V: now also IC2.V-; no longer IC2.V+
- net GND: now also IC2.V+; no longer IC2.V-
Changed lines of the file:
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@@
 <?xml version="1.0" encoding="utf-8"?>
 <!DOCTYPE eagle SYSTEM "eagle.dtd">
-<eagle version="9.0.0">
+<eagle version="9.0.1">
 <drawing>
 <settings>
@@
 <attribute name="OC_MOUSER" value="511-TS507CLT"/>
 </part>
-<part name="GND7" library="supply1" library_urn="urn:adsk.eagle:library:371" deviceset="GND" device=""/>
 <part name="GND8" library="supply1" library_urn="urn:adsk.eagle:library:371" deviceset="GND" device=""/>
 <part name="P+5" library="supply1" library_urn="urn:adsk.eagle:library:371" deviceset="+5V" device=""/>
-<part name="P+6" library="supply1" library_urn="urn:adsk.eagle:library:371" deviceset="+5V" device=""/>
 <part name="GND2" library="supply1" library_urn="urn:adsk.eagle:library:371" deviceset="GND" device=""/>
 <part name="P+7" library="supply1" library_urn="urn:adsk.eagle:library:371" deviceset="+5V" device=""/>
@@
 <part name="P+9" library="supply1" library_urn="urn:adsk.eagle:library:371" deviceset="+5V" device=""/>
 <part name="GND10" library="supply1" library_urn="urn:adsk.eagle:library:371" deviceset="GND" device=""/>
+<part name="P+6" library="supply1" library_urn="urn:adsk.eagle:library:371" deviceset="+5V" device=""/>
+<part name="GND7" library="supply1" library_urn="urn:adsk.eagle:library:371" deviceset="GND" device=""/>
 </parts>
 <sheets>
@@
 <attribute name="OC_MOUSER" x="91.44" y="114.3" size="1.778" layer="96" display="off"/>
 </instance>
-<instance part="GND7" gate="1" x="91.44" y="101.6"/>
 <instance part="GND8" gate="1" x="60.96" y="99.06"/>
 <instance part="P+5" gate="1" x="60.96" y="137.16"/>
-<instance part="P+6" gate="1" x="91.44" y="134.62"/>
 <instance part="GND2" gate="1" x="160.02" y="121.92"/>
 <instance part="P+7" gate="1" x="205.74" y="154.94"/>
@@
 <instance part="P+9" gate="1" x="172.72" y="99.06"/>
 <instance part="GND10" gate="1" x="137.16" y="73.66"/>
+<instance part="P+6" gate="1" x="91.44" y="101.6" rot="R180"/>
+<instance part="GND7" gate="1" x="91.44" y="132.08" rot="R180"/>
 </instances>
 <busses>
@@
 <wire x1="109.22" y1="86.36" x2="109.22" y2="78.74" width="0.1524" layer="91"/>
 <pinref part="GND6" gate="1" pin="GND"/>
-</segment>
-<segment>
-<pinref part="GND7" gate="1" pin="GND"/>
-<pinref part="IC2" gate="G$1" pin="V-"/>
-<wire x1="91.44" y1="104.14" x2="91.44" y2="106.68" width="0.1524" layer="91"/>
 </segment>
 <segment>
@@
 <wire x1="137.16" y1="86.36" x2="147.32" y2="86.36" width="0.1524" layer="91"/>
 </segment>
+<segment>
+<pinref part="IC2" gate="G$1" pin="V+"/>
+<wire x1="91.44" y1="121.92" x2="91.44" y2="129.54" width="0.1524" layer="91"/>
+<pinref part="GND7" gate="1" pin="GND"/>
+</segment>
 </net>
 <net name="AD_COMP" class="0">
@@
 </segment>
 <segment>
-<pinref part="IC2" gate="G$1" pin="V+"/>
-<pinref part="P+6" gate="1" pin="+5V"/>
-<wire x1="91.44" y1="121.92" x2="91.44" y2="132.08" width="0.1524" layer="91"/>
-</segment>
-<segment>
 <wire x1="195.58" y1="142.24" x2="205.74" y2="142.24" width="0.1524" layer="91"/>
 <wire x1="205.74" y1="142.24" x2="205.74" y2="152.4" width="0.1524" layer="91"/>
@@
 <junction x="172.72" y="91.44"/>
 </segment>
+<segment>
+<pinref part="IC2" gate="G$1" pin="V-"/>
+<wire x1="91.44" y1="106.68" x2="91.44" y2="104.14" width="0.1524" layer="91"/>
+<pinref part="P+6" gate="1" pin="+5V"/>
+</segment>
 </net>

Commit message: fixing op amp (iron,tweezer)
Connections:
- net +5V: now also IC2.V+; no longer IC2.V-
- net GND: now also IC2.V-; no longer IC2.V+
Changed lines of the file:
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@@
 <attribute name="OC_MOUSER" value="756-PCF0805R20KBI"/>
 </part>
-<part name="R2" library="solderpi" library_urn="urn:adsk.eagle:library:1437534" deviceset="NTC-0805" device="" package3d_urn="urn:adsk.eagle:package:1581953/2" value="68k @25°C, 1%, ß=4100 K"/>
+<part name="R2" library="solderpi" library_urn="urn:adsk.eagle:library:1437534" deviceset="NTC-0805" device="" package3d_urn="urn:adsk.eagle:package:1581953/4" value="68k @25°C, 1%, ß=4100 K"/>
 <part name="P+1" library="supply1" library_urn="urn:adsk.eagle:library:371" deviceset="+5V" device=""/>
 <part name="GND3" library="supply1" library_urn="urn:adsk.eagle:library:371" deviceset="GND" device=""/>
@@
 </part>
 <part name="GND6" library="supply1" library_urn="urn:adsk.eagle:library:371" deviceset="GND" device=""/>
-<part name="IC2" library="solderpi" library_urn="urn:adsk.eagle:library:1437534" deviceset="TS507CLT" device="" package3d_urn="urn:adsk.eagle:package:1437676/4">
+<part name="IC2" library="solderpi" library_urn="urn:adsk.eagle:library:1437534" deviceset="TS507CLT" device="" package3d_urn="urn:adsk.eagle:package:1437676/7">
 <attribute name="OC_MOUSER" value="511-TS507CLT"/>
 </part>
@@
 <part name="SDA" library="solderpi" library_urn="urn:adsk.eagle:library:1437534" deviceset="1,6/0,8" device="" package3d_urn="urn:adsk.eagle:package:1581957/6"/>
 <part name="+5V" library="solderpi" library_urn="urn:adsk.eagle:library:1437534" deviceset="1,6/0,8" device="" package3d_urn="urn:adsk.eagle:package:1581957/6"/>
-<part name="IC1" library="solderpi" library_urn="urn:adsk.eagle:library:1437534" deviceset="AT24CS04-SOT23" device="" package3d_urn="urn:adsk.eagle:package:1437676/4">
+<part name="IC1" library="solderpi" library_urn="urn:adsk.eagle:library:1437534" deviceset="AT24CS04-SOT23" device="" package3d_urn="urn:adsk.eagle:package:1437676/7">
 <attribute name="OC_MOUSER" value="556-AT24CS04-STUM-T"/>
 </part>
-<part name="IC4" library="solderpi" library_urn="urn:adsk.eagle:library:1437534" deviceset="ESDA6V1SC5" device="" package3d_urn="urn:adsk.eagle:package:1437676/4"/>
+<part name="IC4" library="solderpi" library_urn="urn:adsk.eagle:library:1437534" deviceset="ESDA6V1SC5" device="" package3d_urn="urn:adsk.eagle:package:1437676/7"/>
 <part name="P+9" library="supply1" library_urn="urn:adsk.eagle:library:371" deviceset="+5V" device=""/>
 <part name="GND10" library="supply1" library_urn="urn:adsk.eagle:library:371" deviceset="GND" device=""/>
+<part name="GND7" library="supply1" library_urn="urn:adsk.eagle:library:371" deviceset="GND" device=""/>
 <part name="P+6" library="supply1" library_urn="urn:adsk.eagle:library:371" deviceset="+5V" device=""/>
-<part name="GND7" library="supply1" library_urn="urn:adsk.eagle:library:371" deviceset="GND" device=""/>
 </parts>
 <sheets>
@@
 <instance part="P+9" gate="1" x="172.72" y="99.06"/>
 <instance part="GND10" gate="1" x="137.16" y="73.66"/>
-<instance part="P+6" gate="1" x="91.44" y="101.6" rot="R180"/>
-<instance part="GND7" gate="1" x="91.44" y="132.08" rot="R180"/>
+<instance part="GND7" gate="1" x="91.44" y="101.6"/>
+<instance part="P+6" gate="1" x="91.44" y="129.54"/>
 </instances>
 <busses>
@@
 </segment>
 <segment>
-<pinref part="IC2" gate="G$1" pin="V+"/>
-<wire x1="91.44" y1="121.92" x2="91.44" y2="129.54" width="0.1524" layer="91"/>
 <pinref part="GND7" gate="1" pin="GND"/>
+<pinref part="IC2" gate="G$1" pin="V-"/>
+<wire x1="91.44" y1="104.14" x2="91.44" y2="106.68" width="0.1524" layer="91"/>
 </segment>
 </net>
@@
 </segment>
 <segment>
-<pinref part="IC2" gate="G$1" pin="V-"/>
-<wire x1="91.44" y1="106.68" x2="91.44" y2="104.14" width="0.1524" layer="91"/>
+<pinref part="IC2" gate="G$1" pin="V+"/>
 <pinref part="P+6" gate="1" pin="+5V"/>
+<wire x1="91.44" y1="121.92" x2="91.44" y2="127" width="0.1524" layer="91"/>
 </segment>
 </net>

Commit message: iron drills deleted
Connections:
- net AD_MOTION: now also IC3.VIN0; no longer IC3.VIN2
- net AD_TC: now also IC3.VIN2; no longer IC3.VIN0

Commit message: parts reworked
Parts:
- C1, C2: device rcl:C-EUC0805 -> common:C-EU0603
- IC1: OC_DIGIKEY (none) -> AT24CS04-STUM-TCT-ND; OC_MOUSER 556-AT24CS04-STUM-T -> (none)
- IC2: OC_DIGIKEY (none) -> TS507CLT; OC_MOUSER 511-TS507CLT -> (none)
- IC3: OC_DIGIKEY (none) -> AD7995YRJZ-0500RL7CT-ND; OC_MOUSER 584-AD7995YRJZ0500R7 -> (none)
- IC4: OC_DIGIKEY (none) -> 497-7748-1-ND
- R1: device rcl:R-EU_R0805 -> common:R-EU0603; OC_DIGIKEY (none) -> P20KDBCT-ND; OC_MOUSER 756-PCF0805R20KBI -> (none)
- R10: value 2k 0,1% -> 2k 0.1%; device rcl:R-EU_R0805 -> common:R-EU0603; OC_DIGIKEY (none) -> TNP2.00KAACT-ND; OC_MOUSER 279-RN73C2A2K0BTD -> (none)
- R2: value 68k @25°C, 1%, ß=4100 K -> 68k @25°C, 1%, ß=3985 K; device solderpi:NTC-0805 -> common:NTC0603; OC_DIGIKEY (none) -> BC2555CT-ND
- R4: device rcl:R-EU_R0805 -> common:R-EU0603
- R5, R6: device rcl:R-EU_R0805 -> common:R-EU0603; OC_DIGIKEY (none) -> RMCF0603FT1K00CT-ND; OC_MOUSER 71-CRCW08051K00FKEAC -> (none)
- R7: device rcl:R-EU_R0805 -> common:R-EU0603; OC_DIGIKEY (none) -> TNP2.00KAACT-ND; OC_MOUSER 279-RN73C2A2K0BTD -> (none)
- R8, R9: device rcl:R-EU_R0805 -> common:R-EU0603; OC_DIGIKEY (none) -> YAG4498CT-ND; OC_MOUSER 603-RT0805BRD071ML -> (none)
- renumbered HEATER to PWR
