File: pcb/controller.sch (EAGLE design)
At the start: 167 parts, among them CON1 BINDER-IP40, CON2 BINDER-IP40, IC1 LTC4357, IC10 ST2378E, IC11 5k, IC12 LT1803, IC13 INA196, IC14 INA196, IC15 INA196, IC16 INA196, IC17 INA196, IC18 INA196, IC2 LM1084, IC3 LMR62014, IC4 LM74670, IC5 LM74670, IC6 LM74670, IC7 LM74670, IC8 ATSAMC21J, IC9 PCA9533, Q1 24MHz, Q2 32768kHz, T1 FDS6670A, T10 NVR4003NT3G, T11 NVR4003NT3G, T12 IRF9392PBF, T13 IRF9392PBF, T14 NVR4003NT3G, T15 IRF9392PBF, T16 NVR4003NT3G, T17 IRF9392PBF, T18 BSS7728NH6327XTSA1, T19 BSS84PH6433XTMA1, T2 PSMN1R0, T20 BSS84PH6433XTMA1, T21 BSS84PH6433XTMA1, T3 PSMN1R0, T4 PSMN1R0, T5 PSMN1R0, T6 NVR4003NT3G, T7 NVR4003NT3G, T8 IRF9392PBF, T9 IRF9392PBF, X1 ULTRAFIT-20, X10 IGRID-14, X11 MICRO-CLASP-6, X2 NANOFIT-7, X3 NANOFIT-7, X4 NANOFIT-7, X5 JTAG-EDGE-CON, X6 B3S-1000, X7 IGRID-10, X9 MICRO-LATCH-4

Commit message: initial Commit controller Board
Parts:
- removed C15, C16, C17, C18: 100nF, rcl:C-EUC0402
- removed C19, C20: 27pF, rcl:C-EUC0402
- removed C21, C23: 22pF, rcl:C-EUC0402
- removed C22: 100pF, rcl:C-EUC0603
- removed C24, C25: 100nF, rcl:C-EUC0603
- removed C26, C27, C28, C32, C33, C34: 1nF, rcl:C-EUC0603
- removed C29, C30, C31, C35, C36, C37: 150nF, rcl:C-EUC0603
- removed C38, C39: 10µF, rcl:C-EUC0805
- removed CON1, CON2: BINDER-IP40, solderpi:BINDER-IP40
- removed D1: MBR05020L, solderpi:MBR05020L
- removed IC10: ST2378E, solderpi:ST2378E
- removed IC11: 5k, solderpi:AD5247BKSZ5-RL7
- removed IC12: LT1803, solderpi:LT1803
- removed IC13, IC14, IC15, IC16, IC17, IC18: INA196, solderpi:INA196
- removed IC19: (no value), solderpi:MIC5504
- removed IC4, IC5, IC7: LM74670, solderpi:LM74670
- removed IC8: ATSAMC21J, solderpi:ATSAMC21J
- removed IC9: PCA9533, solderpi:PCA9533
- removed JP1: (no value), solderpi:PINHD-1X6
- removed L1: 10µH, solderpi:WE-TPC
- removed L2: 50R @ 20MHz, solderpi:L-0603
- removed Q1: 24MHz, solderpi:7A-SERIES
- removed Q2: 32768kHz, solderpi:9HT11
- removed R15, R16: 4,7k, rcl:R-EU_R0805
- removed R43, R53, R54, R55: 1k1, rcl:R-EU_R0603
- removed R44, R46, R48: 665k, rcl:R-EU_R0603
- removed R45, R47, R49: 210k, rcl:R-EU_R0603
- removed R50, R51, R52: 20m, rcl:R-EU_R1206
- removed R56, R57, R58, R59, R60, R61, R62, R63: 4.7k, rcl:R-EU_R0603
- removed T1: FDS6670A, solderpi:FDS6670A
- removed T13, T15, T17: IRF9392PBF, solderpi:IRF9392PBF
- removed T14, T16: NVR4003NT3G, solderpi:NVR4003NT3G
- removed T18: BSS7728NH6327XTSA1, solderpi:BSS7728NH6327XTSA1
- removed T19, T20, T21: BSS84PH6433XTMA1, solderpi:BSS84PH6433XTMA1
- removed T2, T3, T4: PSMN1R0, solderpi:PSMN1R0
- removed X10: IGRID-14, solderpi:IGRID-14
- removed X11: MICRO-CLASP-6, solderpi:MICRO-CLASP-6
- removed X12, X13, X14, X15, X16, X17: (no value), solderpi:PINHD-1X2
- removed X5: JTAG-EDGE-CON, solderpi:JTAG-EDGE-CON
- removed X6: B3S-1000, solderpi:B3S-1000
- removed X7: IGRID-10, solderpi:IGRID-10
- removed X8: (no value), con-molex:KK-156-2
- removed X9: MICRO-LATCH-4, solderpi:MICRO-LATCH-4
- added CON3, CON4: BINDER-IP40, solderpi:BINDER-IP40
- added SW1, SW2: EC12E_SW, switch-alps:EC12E_SW
- C10: value 680nF 5% -> 150nF; device rcl:C-EUC0805 -> rcl:C-EUC0603; OC_MOUSER 81-GRM219R71C684JA1D -> 810-C1608X5R1E154K
- C11: value 1µF -> 1nF; device rcl:C-EUC0402 -> rcl:C-EUC0603; OC_MOUSER 81-GRM155R61C105MA2D -> 710-885012206059
- C12: value 100nF -> 150nF; device rcl:C-EUC0402 -> rcl:C-EUC0603; OC_MOUSER 710-885012105016 -> 810-C1608X5R1E154K
- C13: value 100nF -> 10nF; device rcl:C-EUC0402 -> rcl:C-EUC0805; OC_MOUSER 710-885012105016 -> 710-885012207072
- C14: value 10µF -> 1µF; OC_MOUSER 581-0805YD106MAT2A -> 80-C0805C105M3R
- C2, C4: value 3300µ -> 150nF; device solderpi:C-EEVFK -> rcl:C-EUC0603; OC_MOUSER 667-EEV-FK1E332M -> 810-C1608X5R1E154K
- C3: value 2.2µF -> 1nF; device rcl:C-EUC0805 -> rcl:C-EUC0603; OC_MOUSER 603-CC805KKX5R8BB225 -> 710-885012206059
- C5: value 150pF -> 1nF; device rcl:C-EUC0805 -> rcl:C-EUC0603; OC_MOUSER 963-QMK212SD151KD-T -> 710-885012206059
- C6: value 4.7µF -> 10nF; OC_MOUSER 963-TMK212ABJ475MG-T -> 710-885012207072
- C7, C9: value 680nF 5% -> 10nF; OC_MOUSER 81-GRM219R71C684JA1D -> 710-885012207072
- C8: value 680nF 5% -> 1µF; OC_MOUSER 81-GRM219R71C684JA1D -> 80-C0805C105M3R
- IC1: value LTC4357 -> INA196; device solderpi:LTC4357 -> solderpi:INA196; OC_MOUSER 584-LTC4357CMS8#PBF -> 595-INA196AIDBVT
- IC2: value LM1084 -> INA196; device solderpi:LM1084 -> solderpi:INA196; OC_MOUSER 926-LM1084ISX50NOPB -> 595-INA196AIDBVT
- IC3: value LMR62014 -> INA196; device solderpi:LMR62014 -> solderpi:INA196; OC_MOUSER 926-LMR62014XMFENOPB -> 595-INA196AIDBVT
- IC6: value LM74670 -> INA196; device solderpi:LM74670 -> solderpi:INA196; OC_MOUSER 595-LM74670QDGKRQ1 -> 595-INA196AIDBVT
- R1: value 665k -> 4,7k; device rcl:R-EU_R0603 -> rcl:R-EU_R0805; OC_MOUSER 71-CRCW0603-665K-E3 -> 652-CR0805-FX4701GLF
- R10, R12, R13, R14, R5, R6, R7, R9: value 4,7k -> 10k; OC_MOUSER 652-CR0805-FX4701GLF -> 603-RC0805FR-0710KL
- R11, R8: value 4,7k -> 22k; OC_MOUSER 652-CR0805-FX4701GLF -> 603-RC0805FR-0722KL
- R17: value 0 -> 665k; device rcl:R-EU_R1210 -> rcl:R-EU_R0603; OC_MOUSER 603-AC1210JR-070RL -> 71-CRCW0603-665K-E3
- R18, R22: value 10k -> 210k; OC_MOUSER 603-RC0603FR-0710KL -> 603-RC0603FR-10220KL
- R19: value 2k2 -> 20m; device rcl:R-EU_R0603 -> rcl:R-EU_R1206; OC_DIGIKEY (none) -> https://www.digikey.de/product-detail/de/stackpole-electron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; OC_MOUSER 603-RC0603FR-072K2L -> (none)
- R2: value 210k -> 4,7k; device rcl:R-EU_R0603 -> rcl:R-EU_R0805; OC_MOUSER 603-RC0603FR-10220KL -> 652-CR0805-FX4701GLF
- R20: value 330 -> 1k1; OC_MOUSER 594-MCT06030C3300FP5 -> 603-AC0603FR-071K1L
- R21: value 10k -> 665k; OC_MOUSER 603-RC0603FR-0710KL -> 71-CRCW0603-665K-E3
- R23: value 294 -> 20m; device rcl:R-EU_R0805 -> rcl:R-EU_R1206; OC_DIGIKEY (none) -> https://www.digikey.de/product-detail/de/stackpole-electron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; OC_MOUSER 71-CRCW0805-294-E3 -> (none)
- R24: value 10k -> 1k1; OC_MOUSER 603-RC0603FR-0710KL -> 603-AC0603FR-071K1L
- R25: value 100k 0.1% -> 4,7k; device rcl:R-EU_R0603 -> rcl:R-EU_R0805; OC_MOUSER 284-APC0805B100KN -> 652-CR0805-FX4701GLF
- R26: value 41k7 0.1% -> 4,7k; device rcl:R-EU_R0603 -> rcl:R-EU_R0805; OC_MOUSER 71-TNPW080541K7BEEA -> 652-CR0805-FX4701GLF
- R27: value 24k 0.1% -> 4.7k; OC_MOUSER 279-CPF0805B24KE1 -> 603-RC0603FR-0710KL
- R28: value 200 0.1% -> 4.7k; OC_MOUSER 284-APC0805B200RN -> 603-RC0603FR-0710KL
- R29: value 210 -> 4,7k; OC_MOUSER 603-RC0805FR-07210RL -> 652-CR0805-FX4701GLF
- R3: value 13k3 -> 10k; OC_MOUSER 652-CR0805FX-1332ELF -> 603-RC0805FR-0710KL
- R30: value 10k -> 4,7k; device rcl:R-EU_R0603 -> rcl:R-EU_R0805; OC_MOUSER 603-RC0603FR-0710KL -> 652-CR0805-FX4701GLF
- R31: value 210 -> 30k; device rcl:R-EU_R0805 -> rcl:R-EU_R0603; OC_MOUSER 603-RC0805FR-07210RL -> 71-CRCW0603-665K-E3
- R32: value 665k -> 10k; OC_MOUSER 71-CRCW0603-665K-E3 -> 603-RC0603FR-10220KL
- R33, R37: value 210k -> 20m; device rcl:R-EU_R0603 -> rcl:R-EU_R1206; OC_DIGIKEY (none) -> https://www.digikey.de/product-detail/de/stackpole-electron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; OC_MOUSER 603-RC0603FR-10220KL -> (none)
- R34: value 665k -> 1k1; OC_MOUSER 71-CRCW0603-665K-E3 -> 603-AC0603FR-071K1L
- R35: value 210k -> 665k; OC_MOUSER 603-RC0603FR-10220KL -> 71-CRCW0603-665K-E3
- R36: value 665k -> 210k; OC_MOUSER 71-CRCW0603-665K-E3 -> 603-RC0603FR-10220KL
- R38: value 20m -> 1k1; device rcl:R-EU_R1206 -> rcl:R-EU_R0603; OC_MOUSER 791-WW12DR020FTL -> 603-AC0603FR-071K1L
- R39, R40: value 20m -> 4,7k; device rcl:R-EU_R1206 -> rcl:R-EU_R0805; OC_MOUSER 791-WW12DR020FTL -> 652-CR0805-FX4701GLF
- R4: value 182k -> 10k; OC_MOUSER 71-CRCW0805-182K-E3 -> 603-RC0805FR-0710KL
- R41, R42: value 1k1 -> 4.7k; OC_MOUSER 603-AC0603FR-071K1L -> 603-RC0603FR-0710KL
- T11, T7: value NVR4003NT3G -> IRF9392PBF; device solderpi:NVR4003NT3G -> solderpi:IRF9392PBF; OC_MOUSER 863-NVR4003NT3G -> 942-IRF9392TRPBF
- T5: value PSMN1R0 -> NVR4003NT3G; device solderpi:PSMN1R0 -> solderpi:NVR4003NT3G; OC_MOUSER 771-PSMN1R0-30YLDX -> 863-NVR4003NT3G
- T9: value IRF9392PBF -> NVR4003NT3G; device solderpi:IRF9392PBF -> solderpi:NVR4003NT3G; OC_MOUSER 942-IRF9392TRPBF -> 863-NVR4003NT3G
- X1: value ULTRAFIT-20 -> NANOFIT-7; device solderpi:ULTRAFIT-20 -> solderpi:NANOFIT-7; OC_MOUSER 538-172286-1102, 538-172256-2102 -> 538-105313-1107, 538-105307-1207
- X2, X4: value NANOFIT-7 -> PINHD-1X2; device solderpi:NANOFIT-7 -> solderpi:PINHD-1X2; OC_MOUSER 538-105313-1107, 538-105307-1207 -> 855-M20-9990246
Connections:
- removed net +12V_PULSE: IC1.IN, IC4.CATHODE, IC6.CATHODE, JP1.2, R1.2, R25.2, T1.S, T12.S, T13.S, T15.S, T17.S, T2.D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
- removed net +18V: C5.1, C6.1, D1.C, JP1.3, R11.2, R12.2, R14.2, R16.2, R4.2, R7.2, R8.2
- removed net +3V3: C38.1, IC10.OE, IC10.VL, IC19.OUT, JP1.6, X7.7
- removed net 12V_WAVE: C1.1, IC8G$1.PA06, R1.1, R2.2
- removed net AC_IN_+: IC4.ANODE, IC5.CATHODE, T2.S, T3.D, X1.1
- removed net AC_IN_-: IC6.ANODE, IC7.CATHODE, T4.S, T5.D, X1.2
- removed net AGND: C1.2, C13.2, C14.2, C26.2, C27.2, C28.2, C29.2, C30.2, C31.2, C32.2, C33.2, C34.2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
- removed net BOOST_FB: C5.2, IC3.FB, R3.2, R4.1
- removed net BOOST_SW: D1.A, IC3.SW, L1.1
- removed net CON1_HEATER_0: IC14.VIN-, R39.2, X3.1
- removed net CON1_HEATER_0_CUR: C30.1, IC8G$1.PB04, R42.2
- removed net CON1_HEATER_0_IN: IC14.VIN+, R34.2, R39.1, T15.D
- removed net CON1_HEATER_0_VOL: C27.1, IC8G$1.PB05, R34.1, R35.2
- removed net CON1_HEATER_1: IC17.VIN-, R51.2, X3.2
- removed net CON1_HEATER_1_CUR: C36.1, IC8G$1.PB07, R54.2
- removed net CON1_HEATER_1_IN: IC17.VIN+, R46.2, R51.1, T17.D
- removed net CON1_HEATER_1_VOL: C33.1, IC8G$1.PB06, R46.1, R47.2
- removed net CON1_SCL: IC8G$1.PB13, R57.1, X13.2, X3.4
- removed net CON1_SDA: IC8G$1.PB12, R56.1, X13.1, X3.5
- removed net CON2_HEATER_0: IC15.VIN-, R40.2, X4.1
- removed net CON2_HEATER_0_CUR: C31.1, IC8G$2.PB00, R43.2
- removed net CON2_HEATER_0_IN: IC15.VIN+, R36.2, R40.1, T9.D
- removed net CON2_HEATER_0_VOL: C28.1, IC8G$2.PB01, R36.1, R37.2
- removed net CON2_HEATER_1: IC18.VIN-, R52.2, X4.2
- removed net CON2_HEATER_1_CUR: C37.1, IC8G$2.PB03, R55.2
- removed net CON2_HEATER_1_IN: IC18.VIN+, R48.2, R52.1, T13.D
- removed net CON2_HEATER_1_VOL: C34.1, IC8G$2.PB02, R48.1, R49.2
- removed net CON2_SCL: IC8G$2.PB31, R59.1, X15.2, X4.4
- removed net CON2_SDA: IC8G$2.PB30, R58.1, X15.1, X4.5
- removed net DIODE_G: IC1.GATE, T1.G
- removed net HEATER0_AD_OUT0: IC13.VOUT, R41.1
- removed net HEATER0_AD_OUT1: IC16.VOUT, R53.1
- removed net HEATER0_G0: R7.1, T6.D, T8.G
- removed net HEATER0_G1: R11.1, T10.D, T12.G
- removed net HEATER1_AD_OUT0: IC14.VOUT, R42.1
- removed net HEATER1_AD_OUT1: IC17.VOUT, R54.1
- removed net HEATER1_G0: R14.1, T14.D, T15.G
- removed net HEATER1_G1: R16.1, T16.D, T17.G
- removed net HEATER2_AD_OUT0: IC15.VOUT, R43.1
- removed net HEATER2_AD_OUT1: IC18.VOUT, R55.1
- removed net HEATER2_G0: R8.1, T7.D, T9.G
- removed net HEATER2_G1: R12.1, T11.D, T13.G
- removed net HEATER_CTRL_2: IC8G$2.PB22, R13.2, T14.G
- removed net HEATER_CTRL_3: IC8G$2.PB23, R15.2, T16.G
- removed net HEATER_CTRL_4: IC8G$2.PA27, R6.2, T7.G
- removed net HEATER_CTRL_5: IC8G$2.PA28, R10.2, T11.G
- removed net LDO_IN: C2.+, IC1.OUT, IC1.VDD, IC2.IN, T1.D
- removed net LED_BLUE_D: R23.1, T19.D
- removed net LED_BLUE_PWM: IC9.LED1, R22.1, T19.G
- removed net LED_GREEN_D: R31.1, T21.D
- removed net LED_GREEN_PWM: IC9.LED2, R30.1, T21.G
- removed net LED_RED_D: R29.1, T20.D
- removed net LED_RED_PWM: IC9.LED0, R24.1, T20.G
- removed net RECT_D1_CAP_H1: C7.1, IC4.VCAP_H
- removed net RECT_D1_CAP_L1: C7.2, IC4.VCAP_L
- removed net RECT_D1_G1: IC4.G_DRIVE, IC4.G_PULL, T2.G
- removed net RECT_D2_CAP_H1: C9.2, IC6.VCAP_L
- removed net RECT_D2_CAP_L1: C9.1, IC6.VCAP_H
- removed net RECT_D2_G1: IC6.G_DRIVE, IC6.G_PULL, T4.G
- removed net RECT_D3_CAP_H1: C8.1, IC5.VCAP_H
- removed net RECT_D3_CAP_L1: C8.2, IC5.VCAP_L
- removed net RECT_D3_G1: IC5.G_DRIVE, IC5.G_PULL, T3.G
- removed net RECT_D4_CAP_H1: C10.2, IC7.VCAP_L
- removed net RECT_D4_CAP_L1: C10.1, IC7.VCAP_H
- removed net RECT_D4_G1: IC7.G_DRIVE, IC7.G_PULL, T5.G
- removed net RESETN: C22.2, IC10.IO_VCC_7, IC8G$3.RESETN, R19.1, R20.2, X5.10
- removed net RESET_SW_IN: R20.1, X6.S
- removed net RPI_HARDRST_1: T18.D, X7.9
- removed net RPI_HARDRST_2: T18.S, X7.10
- removed net RPI_INT: IC10.IO_VL_8, X7.5
- removed net RPI_INT_HI: IC10.IO_VCC_8, IC8G$2.PA20
- removed net RPI_RESET: IC8G$1.PA03, R21.2, T18.G
- removed net RPI_RXD: IC10.IO_VL_3, X17.1, X7.2
- removed net RPI_RXD_HI: IC10.IO_VCC_3, IC8G$2.PA17, X14.1
- removed net RPI_SWCLK: IC10.IO_VL_6, X7.3
- removed net RPI_SWDIO: IC10.IO_VL_5, X7.4
- removed net RPI_SWRST: IC10.IO_VL_7, X7.6
- removed net RPI_TXD: IC10.IO_VL_4, X17.2, X7.1
- removed net RPI_TXD_HI: IC10.IO_VCC_4, IC8G$2.PA16, X14.2
- removed net SWCLK: IC10.IO_VCC_6, IC8G$3.SWCLK, X5.9
- removed net SWDIO: IC10.IO_VCC_5, IC8G$3.SWDIO, X5.6
- removed net UI_BUTTON: IC8G$2.PA21, R18.1, X11.1
- removed net UI_LED_BLUE: R23.2, X11.4
- removed net UI_LED_GREEN: R31.2, X11.3
- removed net UI_LED_RED: R29.2, X11.5
- removed net UI_ROT2_A: IC8G$1.PB14, X10.9
- removed net UI_ROT2_B: IC8G$1.PB10, X10.13
- removed net UI_ROT2_SW: IC8G$1.PB09, X10.11
- removed net UI_ROT3_A: IC8G$2.PB17, X10.1
- removed net UI_ROT3_B: IC8G$1.PA12, X10.5
- removed net UI_ROT3_SW: IC8G$2.PA19, X10.3
- removed net UI_ROT4_A: IC8G$1.PA13, X10.6
- removed net UI_ROT4_B: IC8G$2.PB16, X10.2
- removed net UI_ROT4_SW: IC8G$2.PA18, X10.4
- removed net UI_SCL: IC11G$1.SCL, IC8G$2.PA23, IC9.SCL, R63.1, X16.2, X9.4
- removed net UI_SDA: IC11G$1.SDA, IC8G$2.PA22, IC9.SDA, R62.1, X16.1, X9.3
- removed net VDDANA: C13.1, C14.1, IC8G$4.VDDANA, L2.2
- removed net VDDCORE: C11.1, C12.1, IC8G$4.VDDCORE
- removed net XIN: C19.1, IC8G$4.XIN, Q1.1
- removed net XIN32: C21.1, IC8G$4.XIN32, Q2.1
- removed net XOUT: C20.1, IC8G$4.XOUT, Q1.2
- removed net XOUT32: C23.1, IC8G$4.XOUT32, Q2.2
- removed net ZC_ADJ: IC11G$2.A, IC11G$2.W, R28.1
- removed net ZC_IN+: IC12.+IN, R27.1, R28.2
- removed net ZC_IN+-: IC12.-IN, R25.1, R26.2
- removed net ZERO_CROSSING: IC12.OUT, IC8G$1.PA07, JP1.5
- new net +12V: R2.2, R25.2, R30.2, R39.2, T11.S, T12.S, T7.S, T8.S
- new net 2_HEATER_PI: CON3.P$2
- new net 5_SDA_YE: CON3.P$7
- new net HEATER0_AD_OUT2: IC1.VOUT, R20.1
- new net HEATER0_AD_OUT3: IC2.VOUT, R24.1
- new net HEATER0_AD_OUT4: IC3.VOUT, R34.1
- new net HEATER0_AD_OUT5: IC6.VOUT, R38.1
- new net HEATER0_G2: R25.1, T6.D, T8.G
- new net HEATER0_G3: R2.1, T5.D, T7.G
- new net HEATER0_G4: R39.1, T10.D, T12.G
- new net HEATER0_G5: R30.1, T11.G, T9.D
- new net UI_ROT1_A_UNFIL: R3.1, R4.2, SW1G$1.A
- new net UI_ROT1_A_UNFIL1: R12.2, R6.1, SW2G$1.A
- new net UI_ROT1_B_UNFIL: R5.1, R7.1, SW1G$1.B
- new net UI_ROT1_B_UNFIL1: R10.1, R13.1, SW2G$1.B
- new net UI_ROT1_SW_R: R11.1, R9.1, SW1G$2.1
- new net UI_ROT1_SW_R1: R14.1, R8.1, SW2G$2.1
- new net VCC: IC1.V+, IC2.V+, IC3.V+, IC6.V+
- net +5V: now also R10.2, R14.2, R28.2, R3.2, R41.2, R42.2, R5.2, R6.2, R9.2, X1.3; no longer C15.1, C16.1, C17.1, C18.1, C22.1, C24.1, C25.1, C3.1, C39.1, C4.+, IC10.VCC, IC11G$1.VDD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
- net 1_HEATER1_BR: now also CON3.P$4, CON4.P$4; no longer CON1.1, CON2.1
- net 3_+5V_GY: now also CON3.P$3, CON4.P$3; no longer CON1.3, CON2.3
- net 4_SCL_GR: now also CON3.P$6, CON4.P$6; no longer CON1.4, CON2.4
- net 6_GND_WH: now also CON3.P$5, CON4.P$5; no longer CON1.6, CON2.6
- net 7_GND_BL: now also CON3.P$1; no longer CON1.7
- net CON0_HEATER_0: now also IC1.VIN-, IC3.VIN-, R19.2, R33.2, X1.1, X3.1; no longer IC13.VIN-, R38.2, X2.1
- net CON0_HEATER_0_CUR: now also C10.1, C2.1, R20.2, R34.2; no longer C29.1, IC8G$1.PA04, R41.2
- net CON0_HEATER_0_IN: now also IC1.VIN+, IC3.VIN+, R17.2, R19.1, R31.2, R33.1, T11.D, T7.D; no longer IC13.VIN+, R32.2, R38.1, T8.D
- net CON0_HEATER_0_VOL: now also C1.1, C5.1, R17.1, R18.2, R31.1, R32.2; no longer C26.1, IC8G$1.PA05, R32.1, R33.2
- net CON0_HEATER_1: now also IC2.VIN-, IC6.VIN-, R23.2, R37.2, X1.2, X3.2; no longer IC16.VIN-, R50.2, X2.2
- net CON0_HEATER_1_CUR: now also C12.1, C4.1, R24.2, R38.2; no longer C35.1, IC8G$1.PA11, R53.2
- net CON0_HEATER_1_IN: now also IC2.VIN+, IC6.VIN+, R21.2, R23.1, R35.2, R37.1, T8.D; no longer IC16.VIN+, R44.2, R50.1
- net CON0_HEATER_1_VOL: now also C11.1, C3.1, R21.1, R22.2, R35.1, R36.2; no longer C32.1, IC8G$1.PA10, R44.1, R45.2
- net CON0_SCL: now also R27.1, R41.1, X1.4, X2.1, X3.4; no longer IC8G$1.PA09, R61.1, X12.2, X2.4
- net CON0_SDA: now also R28.1, R42.1, X1.5, X2.2, X3.5; no longer IC8G$1.PA08, R60.1, X12.1, X2.5
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Other:
- note removed: "12V rectified wave 100Hz fg = 1kHz"
- note removed: "AC Input"
- note removed: "AD5247"
- note removed: "AD5247 - 0101110 MCP4018 - 0101111 MCP23017 - 0100000 PCA9533 - 1100010"
- note removed: "ADC0 | AIN[10]"
- note removed: "ADC0 | AIN[11]"
- note removed: "ADC0 | AIN[4]"
- note removed: "ADC0 | AIN[5]"
- note removed: "ADC0 | AIN[6]"
- note removed: "ADC1 | AIN[0]"
- note removed: "ADC1 | AIN[1]"
- note removed: "ADC1 | AIN[2]"
- note removed: "ADC1 | AIN[3]"
- note removed: "ADC1 | AIN[6]"
- note removed: "ADC1 | AIN[7]"
- note removed: "ADC1 | AIN[8]"
- note removed: "ADC1 | AIN[9]"
- note removed: "Boost Converter 5V->18V"
- note removed: "Button Interface"
- note removed: "Button LEDs"
- note removed: "EXINT[0]"
- note removed: "EXINT[10]"
- note removed: "EXINT[11]"
- note removed: "EXINT[12]"
- note removed: "EXINT[13]"
- note removed: "EXINT[14]"
- note removed: "EXINT[15]"
- note removed: "EXINT[1]"
- note removed: "EXINT[2]"
- note removed: "EXINT[3]"
- note removed: "EXINT[4]"
- note removed: "EXINT[5]"
- note removed: "EXINT[7]"
- note removed: "EXINT[8]"
- note removed: "EXINT[9]"
- note removed: "Ideal Bridge Rectifier"
- note removed: "Interrupt 12x rotary encoder ------ 1x button ------ 1x zero crossing detector ------ serial com 4x i2c ------ 1x uart (cts,rts) ------ output 3x pwm led ------ 6x heater ------ input 13x analog ------"
- note removed: "JTAG Connector"
- note removed: "JTAG Interface"
- note removed: "LCD Interface"
- note removed: "LDO 17V -> 5V"
- note removed: "MCU Power Unit"
- note removed: "OUTPUT"
- note removed: "RPI Interface"
- note removed: "RPI Shifter 3V <-> 5V"
- note removed: "RPI Supply"
- note removed: "Rotary Encoder"
- note removed: "SERCOM0 PAD[0]"
- note removed: "SERCOM0 PAD[1]"
- note removed: "SERCOM1 PAD[0]"
- note removed: "SERCOM1 PAD[1]"
- note removed: "SERCOM3 PAD[0]"
- note removed: "SERCOM3 PAD[1]"
- note removed: "SERCOM4 PAD[0]"
- note removed: "SERCOM4 PAD[1]"
- note removed: "SERCOM5 PAD[0]"
- note removed: "SERCOM5 PAD[1]"
- note removed: "Serial Communication Debug-Pins"
- note removed: "Voltage Pins"
- note removed: "Zero Crossing Detector"

Commit message: wip connect mcu
Parts:
- removed R40: 4,7k, rcl:R-EU_R0805
- removed R42: 4.7k, rcl:R-EU_R0603
- removed T10: NVR4003NT3G, solderpi:NVR4003NT3G
- removed T11, T12, T8: IRF9392PBF, solderpi:IRF9392PBF
- added C15, C16, C17, C18: 100nF, rcl:C-EUC0603
- added IC4: INA196, solderpi:INA196
- added IC5: STM32L496X, solderpi:STM32L496X
- added IC7: TPS62162, solderpi:TPS62162
- added L1, L2: (no value), solderpi:VLF3012S
- added L3: 300R @ 100MHz, solderpi:L0603
- added Q1: 24Mhz, solderpi:XRCHA_F_A
- added R15: 1k, rcl:R-EU_R0603
- added R16: 4,7k, rcl:R-EU_R0805
- added SV1: (no value), solderpi:ML20
- added T1, T4: NVR4003NT3G, solderpi:NVR4003NT3G
- added T2, T3: IRF7416, solderpi:IRF7416
- added X5: NEWHAVEN_OLED_256X64, solderpi:NEWHAVEN_OLED_256X64
- added X6: ULTRAFIT-290, solderpi:ULTRAFIT-290
- C1, C3: value 1nF -> 22µ; device rcl:C-EUC0603 -> rcl:C-EUC0805; OC_DIGIKEY (none) -> 1276-6526-1-ND; OC_MOUSER 710-885012206059 -> (none)
- C10: value 150nF -> 1µF; OC_DIGIKEY (none) -> 1276-1034-1-ND; OC_MOUSER 810-C1608X5R1E154K -> (none)
- C11: value 1nF -> 10nF; OC_DIGIKEY (none) -> 478-6209-1-ND; OC_MOUSER 710-885012206059 -> (none)
- C12: value 150nF -> 100nF; OC_DIGIKEY (none) -> 1276-1005-1-ND; OC_MOUSER 810-C1608X5R1E154K -> (none)
- C2, C4: value 150nF -> 10µ; device rcl:C-EUC0603 -> rcl:C-EUC0805; OC_DIGIKEY (none) -> 1276-2890-1-ND; OC_MOUSER 810-C1608X5R1E154K -> (none)
- C5: value 1nF -> 470µF; device rcl:C-EUC0603 -> solderpi:C-EEEFK; OC_MOUSER 710-885012206059 -> 667-EEE-FK1E471P
- IC6: value INA196 -> TPS62173; device solderpi:INA196 -> solderpi:TPS62173; OC_DIGIKEY (none) -> 296-39450-1-ND; OC_MOUSER 595-INA196AIDBVT -> (none)
- R1, R2, R26, R30: OC_DIGIKEY (none) -> CR0805-FX-4701GLFTR-ND; OC_MOUSER 652-CR0805-FX4701GLF -> (none)
- R17: value 665k -> 1k; OC_DIGIKEY (none) -> RMCF0603FT1K00CT-ND; OC_MOUSER 71-CRCW0603-665K-E3 -> (none)
- R18, R22: value 210k -> 30k; OC_DIGIKEY (none) -> RMCF0603FT30K0CT-ND; OC_MOUSER 603-RC0603FR-10220KL -> (none)
- R19, R23: value 20m -> 10k; device rcl:R-EU_R1206 -> rcl:R-EU_R0603; OC_DIGIKEY https://www.digikey.de/product-detail/de/stackpole-electron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 -> RMCF0603FT10K0CT-ND
- R20, R24: value 1k1 -> 20m; device rcl:R-EU_R0603 -> rcl:R-EU_R2010; OC_DIGIKEY (none) -> 541-10266-1-ND; OC_MOUSER 603-AC0603FR-071K1L -> (none)
- R21: value 665k -> 4,7k; device rcl:R-EU_R0603 -> rcl:R-EU_R0805; OC_DIGIKEY (none) -> CR0805-FX-4701GLFTR-ND; OC_MOUSER 71-CRCW0603-665K-E3 -> (none)
- R25, R29: value 4,7k -> 1k; device rcl:R-EU_R0805 -> rcl:R-EU_R0603; OC_DIGIKEY (none) -> RMCF0603FT1K00CT-ND; OC_MOUSER 652-CR0805-FX4701GLF -> (none)
- R27, R28: value 4.7k -> 4,7k; device rcl:R-EU_R0603 -> rcl:R-EU_R0805; OC_DIGIKEY (none) -> CR0805-FX-4701GLFTR-ND; OC_MOUSER 603-RC0603FR-0710KL -> (none)
- R31: OC_DIGIKEY (none) -> RMCF0603FT30K0CT-ND; OC_MOUSER 71-CRCW0603-665K-E3 -> (none)
- R32: OC_DIGIKEY (none) -> RMCF0603FT10K0CT-ND; OC_MOUSER 603-RC0603FR-10220KL -> (none)
- R33: device rcl:R-EU_R1206 -> rcl:R-EU_R2010; OC_DIGIKEY https://www.digikey.de/product-detail/de/stackpole-electron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 -> 541-10266-1-ND
- R34: value 1k1 -> 30k; OC_DIGIKEY (none) -> RMCF0603FT30K0CT-ND; OC_MOUSER 603-AC0603FR-071K1L -> (none)
- R35: value 665k -> 10k; OC_DIGIKEY (none) -> RMCF0603FT10K0CT-ND; OC_MOUSER 71-CRCW0603-665K-E3 -> (none)
- R36: value 210k -> 20m; device rcl:R-EU_R0603 -> rcl:R-EU_R2010; OC_DIGIKEY (none) -> 541-10266-1-ND; OC_MOUSER 603-RC0603FR-10220KL -> (none)
- R37: value 20m -> 100k; device rcl:R-EU_R1206 -> rcl:R-EU_R0603; OC_DIGIKEY https://www.digikey.de/product-detail/de/stackpole-electron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 -> RMCF0603FT100KCT-ND
- R38: value 1k1 -> 100k; OC_DIGIKEY (none) -> RMCF0603FT100KCT-ND; OC_MOUSER 603-AC0603FR-071K1L -> (none)
- R39: value 4,7k -> 0; device rcl:R-EU_R0805 -> rcl:R-EU_R2010; OC_DIGIKEY (none) -> RMCF2010ZT0R00CT-ND; OC_MOUSER 652-CR0805-FX4701GLF -> (none)
- R41: value 4.7k -> 10k; OC_DIGIKEY (none) -> RMCF0603FT10K0CT-ND; OC_MOUSER 603-RC0603FR-0710KL -> (none)
- T5, T9: OC_DIGIKEY (none) -> NVR4003NT3GOSCT-ND; OC_MOUSER 863-NVR4003NT3G -> (none)
- T6: value NVR4003NT3G -> IRF7416; device solderpi:NVR4003NT3G -> solderpi:IRF7416; OC_DIGIKEY (none) -> IRF7416TRPBFCT-ND; OC_MOUSER 863-NVR4003NT3G -> (none)
- T7: value IRF9392PBF -> IRF7416; device solderpi:IRF9392PBF -> solderpi:IRF7416; OC_DIGIKEY (none) -> IRF7416TRPBFCT-ND; OC_MOUSER 942-IRF9392TRPBF -> (none)
Connections:
- net UI_ROT1_A_UNFIL renamed ROT0_A_UNFIL
- net UI_ROT1_A_UNFIL1 renamed ROT1_A_UNFIL
- net UI_ROT1_B_UNFIL renamed ROT0_B_UNFIL
- net UI_ROT1_B_UNFIL1 renamed ROT1_B_UNFIL
- net UI_ROT1_SW_R renamed ROT0_SW_R
- net UI_ROT1_SW_R1 renamed ROT1_SW_R
- removed net CON0_HEATER_0: IC1.VIN-, IC3.VIN-, R19.2, R33.2, X1.1, X3.1
- removed net CON0_HEATER_0_CUR: C10.1, C2.1, R20.2, R34.2
- removed net CON0_HEATER_0_IN: IC1.VIN+, IC3.VIN+, R17.2, R19.1, R31.2, R33.1, T11.D, T7.D
- removed net CON0_HEATER_0_VOL: C1.1, C5.1, R17.1, R18.2, R31.1, R32.2
- removed net CON0_HEATER_1: IC2.VIN-, IC6.VIN-, R23.2, R37.2, X1.2, X3.2
- removed net CON0_HEATER_1_CUR: C12.1, C4.1, R24.2, R38.2
- removed net CON0_HEATER_1_IN: IC2.VIN+, IC6.VIN+, R21.2, R23.1, R35.2, R37.1, T12.D, T8.D
- removed net CON0_HEATER_1_VOL: C11.1, C3.1, R21.1, R22.2, R35.1, R36.2
- removed net CON0_SCL: R27.1, R41.1, X1.4, X2.1, X3.4
- removed net CON0_SDA: R28.1, R42.1, X1.5, X2.2, X3.5
- removed net HEATER0_AD_OUT2: IC1.VOUT, R20.1
- removed net HEATER0_AD_OUT3: IC2.VOUT, R24.1
- removed net HEATER0_AD_OUT4: IC3.VOUT, R34.1
- removed net HEATER0_AD_OUT5: IC6.VOUT, R38.1
- removed net HEATER0_G2: R25.1, T6.D, T8.G
- removed net HEATER0_G3: R2.1, T5.D, T7.G
- removed net HEATER0_G4: R39.1, T10.D, T12.G
- removed net HEATER0_G5: R30.1, T11.G, T9.D
- removed net HEATER_CTRL_0: R1.2, R29.2, T5.G, T9.G
- removed net HEATER_CTRL_1: R26.2, R40.2, T10.G, T6.G
- removed net UI_ROT1_A: C6.1, C9.1, R12.1, R4.1
- removed net UI_ROT1_B: C13.1, C7.1, R13.2, R7.2
- removed net UI_ROT1_SW: C14.1, C8.1, R11.2, R8.2
- removed net VCC: IC1.V+, IC2.V+, IC3.V+, IC6.V+
- new net +3V3: C15.1, C16.1, C17.1, C18.1, C3.1, IC2.V+, IC4.V+, IC5G$3.VDD@1, IC5G$3.VDD@2, IC5G$3.VDD@3, IC5G$3.VDDUSB, IC7.VOS, L2.1, L3.2, R10.2, R14.2, R3.2, R38.2, R5.2, R6.2, R9.2, SV1.1
- new net +3V3_ANA: C10.1, C11.1, C12.1, IC5G$3.VDDA/VREF+
- new net AGND: C10.2, C11.2, C12.2, IC5G$3.VSSA/VREF-, R39.2
- new net N$1: C14.1, R8.2
- new net N$10: IC3.VIN-, R33.2
- new net N$11: IC3.VIN+, R31.2, R33.1
- new net N$12: R31.1, R32.2
- new net N$13: IC1.VIN-, R20.2
- new net N$14: IC1.VIN+, R18.2, R20.1
- new net N$15: X4.2
- new net N$16: X4.1
- new net N$17: R18.1, R19.2
- new net N$18: X2.1
- new net N$19: X2.2
- new net N$2: R15.1, X3.4
- new net N$20: R25.1, X1.4
- new net N$21: R29.1, X1.5
- new net N$22: R28.2, T4.G
- new net N$23: R27.2, T5.G
- new net N$24: R26.1, T5.D, T7.G
- new net N$25: R21.1, T4.D, T6.G
- new net N$26: T7.D
- new net N$27: T6.D
- new net N$28: IC2.VIN-, R24.2
- new net N$29: IC2.VIN+, R22.2, R24.1
- new net N$3: R17.1, X3.5
- new net N$30: R22.1, R23.2
- new net N$31: IC4.VIN-, R36.2
- new net N$32: IC4.VIN+, R34.2, R36.1
- new net N$33: R34.1, R35.2
- new net N$34: X5.VDD
- new net N$35: IC1.V+
- new net N$36: IC3.V+
- new net N$37: IC5G$3.PH3-BOOT0, R41.2
- new net N$39: IC7.SW, L2.2
- new net N$4: R16.2, T9.G
- new net N$40: IC6.SW, L1.2
- new net N$42: IC6.PG, R37.1
- new net N$45: IC7.PG, R38.1
- new net N$5: R2.2, T1.G
- new net N$6: R1.1, T1.D, T2.G
- new net N$7: R30.1, T3.G, T9.D
- new net N$8: T2.D
- new net N$9: T3.D
- new net OLED_!CS: X5.!CS
- new net OLED_!RESET: X5.!RES
- new net OLED_D/C: X5.D/C
- new net OLED_SDCLK: X5.SDCLK
- new net OLED_SDIN: X5.SDIN
- new net OSC_IN: IC5G$1.PH0-OSC_IN, Q1.1
- new net OSC_OUT: IC5G$1.PH1-OSC_OUT, Q1.2
- new net RESET: SV1.15
- new net ROT0_A: C6.1, R4.1
- new net ROT0_B: C7.1, R7.2
- new net ROT1_A: C9.1, R12.1
- new net ROT1_B: C13.1, R13.2
- new net ROT1_SW: C8.1, R11.2
- new net SWDCLK: SV1.9
- new net SWDIO: SV1.7
- new net SWO: SV1.13
- net +12V: now also C2.1, C4.1, C5.+, IC6.EN, IC6.VIN, IC7.EN, IC7.VIN, R1.2, R21.2, R26.2, T2.S, T3.S, T6.S, X6.1; no longer R2.2, R25.2, R39.2, T11.S, T12.S, T8.S
- net +5V: now also C1.1, IC6.VOS, L1.1, R15.2, R17.2, R25.2, R29.2, R37.2; no longer R10.2, R14.2, R27.2, R28.2, R3.2, R41.2, R42.2, R5.2, R6.2, R9.2
- net GND: now also C15.2, C16.2, C17.2, C18.2, C5.-, IC4.GND, IC5G$3.VSS@1, IC5G$3.VSS@2, IC5G$3.VSS@3, IC5G$3.VSS@4, IC6.AGND, IC6.FB, IC6.PGND, IC7.AGND, IC7.FB, IC7.PGND, R16.1, R19.1, R2.1, R23.1, R27.1, R28.1, R35.1, R39.1, R41.1, SV1.10, SV1.12, SV1.4, SV1.6, SV1.8, T1.S, T4.S, X5.BS0, X5.BS1, X5.VSS@1, X5.VSS@2, X5.VSS@3, X5.VSS@4, X5.VSS@5, X5.VSS@6, X5.VSS@7, X5.VSS@8, X6.2; no longer C10.2, C11.2, C12.2, C5.2, IC6.GND, R1.1, R18.1, R22.1, R26.1, R29.1, R36.1, R40.1, T10.S, T6.S

Commit message: circuit fully connected
Parts:
- removed CON3, CON4: BINDER-IP40, solderpi:BINDER-IP40
- removed T9: NVR4003NT3G, solderpi:NVR4003NT3G
- added CON1, CON2: BINDER-IP40, solderpi:BINDER-IP40
- added R40: 10k, rcl:R-EU_R0805
- added R42: 22k, rcl:R-EU_R0805
- added T8: IRF7416, solderpi:IRF7416
- C1, C3: value 22µ -> 100nF; device rcl:C-EUC0805 -> rcl:C-EUC0603; OC_DIGIKEY 1276-6526-1-ND -> 1276-1005-1-ND
- C10: value 1µF -> 470µF; device rcl:C-EUC0603 -> solderpi:C-EEEFK; OC_DIGIKEY 1276-1034-1-ND -> (none); OC_MOUSER (none) -> 667-EEE-FK1E471P
- C11: value 10nF -> 22µ; device rcl:C-EUC0603 -> rcl:C-EUC0805; OC_DIGIKEY 478-6209-1-ND -> 1276-6526-1-ND
- C12: value 100nF -> 22µ; device rcl:C-EUC0603 -> rcl:C-EUC0805; OC_DIGIKEY 1276-1005-1-ND -> 1276-6526-1-ND
- C14: value 1µF -> 10nF; OC_MOUSER 80-C0805C105M3R -> 710-885012207072
- C15, C18: value 100nF -> 1µF; device rcl:C-EUC0603 -> rcl:C-EUC0805; OC_DIGIKEY 1276-1005-1-ND -> (none); OC_MOUSER (none) -> 80-C0805C105M3R
- C16, C17: value 100nF -> 10nF; device rcl:C-EUC0603 -> rcl:C-EUC0805; OC_DIGIKEY 1276-1005-1-ND -> (none); OC_MOUSER (none) -> 710-885012207072
- C2: value 10µ -> 1µF; device rcl:C-EUC0805 -> rcl:C-EUC0603; OC_DIGIKEY 1276-2890-1-ND -> 1276-1034-1-ND
- C4: value 10µ -> 10nF; device rcl:C-EUC0805 -> rcl:C-EUC0603; OC_DIGIKEY 1276-2890-1-ND -> 478-6209-1-ND
- C5: value 470µF -> 100nF; device solderpi:C-EEEFK -> rcl:C-EUC0603; OC_DIGIKEY (none) -> 1276-1005-1-ND; OC_MOUSER 667-EEE-FK1E471P -> (none)
- C6, C7: value 10nF -> 100nF; device rcl:C-EUC0805 -> rcl:C-EUC0603; OC_DIGIKEY (none) -> 1276-1005-1-ND; OC_MOUSER 710-885012207072 -> (none)
- C8: value 1µF -> 10µ; OC_DIGIKEY (none) -> 1276-2890-1-ND; OC_MOUSER 80-C0805C105M3R -> (none)
- C9: value 10nF -> 10µ; OC_DIGIKEY (none) -> 1276-2890-1-ND; OC_MOUSER 710-885012207072 -> (none)
- IC1: value INA196 -> STM32L496X; device solderpi:INA196 -> solderpi:STM32L496X; OC_DIGIKEY (none) -> 497-17173-ND; OC_MOUSER 595-INA196AIDBVT -> (none)
- IC2: value INA196 -> TPS62173; device solderpi:INA196 -> solderpi:TPS62173; OC_DIGIKEY (none) -> 296-39450-1-ND; OC_MOUSER 595-INA196AIDBVT -> (none)
- IC3: value INA196 -> TPS62162; device solderpi:INA196 -> solderpi:TPS62162; OC_DIGIKEY (none) -> 296-29897-1-ND; OC_MOUSER 595-INA196AIDBVT -> (none)
- IC4: OC_DIGIKEY (none) -> 296-17166-1-ND; OC_MOUSER 595-INA196AIDBVT -> (none)
- IC5: value STM32L496X -> INA196; device solderpi:STM32L496X -> solderpi:INA196; OC_DIGIKEY 497-17173-ND -> 296-17166-1-ND
- IC6: value TPS62173 -> INA196; device solderpi:TPS62173 -> solderpi:INA196; OC_DIGIKEY 296-39450-1-ND -> 296-17166-1-ND
- IC7: value TPS62162 -> INA196; device solderpi:TPS62162 -> solderpi:INA196; OC_DIGIKEY 296-29897-1-ND -> 296-17166-1-ND
- R1, R2, R30: value 4,7k -> 10k; device rcl:R-EU_R0805 -> rcl:R-EU_R0603; OC_DIGIKEY CR0805-FX-4701GLFTR-ND -> RMCF0603FT10K0CT-ND
- R10, R7, R9: value 10k -> 4,7k; OC_DIGIKEY (none) -> CR0805-FX-4701GLFTR-ND; OC_MOUSER 603-RC0805FR-0710KL -> (none)
- R11: value 22k -> 30k; device rcl:R-EU_R0805 -> rcl:R-EU_R0603; OC_DIGIKEY (none) -> RMCF0603FT30K0CT-ND; OC_MOUSER 603-RC0805FR-0722KL -> (none)
- R12, R14, R3: device rcl:R-EU_R0805 -> rcl:R-EU_R0603; OC_DIGIKEY (none) -> RMCF0603FT10K0CT-ND; OC_MOUSER 603-RC0805FR-0710KL -> (none)
- R13: value 10k -> 30k; device rcl:R-EU_R0805 -> rcl:R-EU_R0603; OC_DIGIKEY (none) -> RMCF0603FT30K0CT-ND; OC_MOUSER 603-RC0805FR-0710KL -> (none)
- R15: value 1k -> 20m; device rcl:R-EU_R0603 -> rcl:R-EU_R2010; OC_DIGIKEY RMCF0603FT1K00CT-ND -> 541-10266-1-ND
- R16: value 4,7k -> 20m; device rcl:R-EU_R0805 -> rcl:R-EU_R2010; OC_DIGIKEY CR0805-FX-4701GLFTR-ND -> 541-10266-1-ND
- R17: value 1k -> 10k; device rcl:R-EU_R0603 -> rcl:R-EU_R0805; OC_DIGIKEY RMCF0603FT1K00CT-ND -> (none); OC_MOUSER (none) -> 603-RC0805FR-0710KL
- R18, R22: value 30k -> 10k; device rcl:R-EU_R0603 -> rcl:R-EU_R0805; OC_DIGIKEY RMCF0603FT30K0CT-ND -> (none); OC_MOUSER (none) -> 603-RC0805FR-0710KL
- R19: value 10k -> 1k; OC_DIGIKEY RMCF0603FT10K0CT-ND -> RMCF0603FT1K00CT-ND
- R20: value 20m -> 10k; device rcl:R-EU_R2010 -> rcl:R-EU_R0805; OC_DIGIKEY 541-10266-1-ND -> (none); OC_MOUSER (none) -> 603-RC0805FR-0710KL
- R21: value 4,7k -> 1k; device rcl:R-EU_R0805 -> rcl:R-EU_R0603; OC_DIGIKEY CR0805-FX-4701GLFTR-ND -> RMCF0603FT1K00CT-ND
- R23, R35, R41: device rcl:R-EU_R0603 -> rcl:R-EU_R0805; OC_DIGIKEY RMCF0603FT10K0CT-ND -> (none); OC_MOUSER (none) -> 603-RC0805FR-0710KL
- R24: value 20m -> 22k; device rcl:R-EU_R2010 -> rcl:R-EU_R0805; OC_DIGIKEY 541-10266-1-ND -> (none); OC_MOUSER (none) -> 603-RC0805FR-0722KL
- R25: value 1k -> 4,7k; device rcl:R-EU_R0603 -> rcl:R-EU_R0805; OC_DIGIKEY RMCF0603FT1K00CT-ND -> CR0805-FX-4701GLFTR-ND
- R29: value 1k -> 30k; OC_DIGIKEY RMCF0603FT1K00CT-ND -> RMCF0603FT30K0CT-ND
- R34: value 30k -> 20m; device rcl:R-EU_R0603 -> rcl:R-EU_R2010; OC_DIGIKEY RMCF0603FT30K0CT-ND -> 541-10266-1-ND
- R36: value 20m -> 1k; device rcl:R-EU_R2010 -> rcl:R-EU_R0603; OC_DIGIKEY 541-10266-1-ND -> RMCF0603FT1K00CT-ND
- R37: value 100k -> 10k; device rcl:R-EU_R0603 -> rcl:R-EU_R0805; OC_DIGIKEY RMCF0603FT100KCT-ND -> (none); OC_MOUSER (none) -> 603-RC0805FR-0710KL
- R38: value 100k -> 1k; OC_DIGIKEY RMCF0603FT100KCT-ND -> RMCF0603FT1K00CT-ND
- R39: value 0 -> 10k; device rcl:R-EU_R2010 -> rcl:R-EU_R0805; OC_DIGIKEY RMCF2010ZT0R00CT-ND -> (none); OC_MOUSER (none) -> 603-RC0805FR-0710KL
- R4, R5: value 10k -> 100k; device rcl:R-EU_R0805 -> rcl:R-EU_R0603; OC_DIGIKEY (none) -> RMCF0603FT100KCT-ND; OC_MOUSER 603-RC0805FR-0710KL -> (none)
- R6: value 10k -> 0; device rcl:R-EU_R0805 -> rcl:R-EU_R2010; OC_DIGIKEY (none) -> RMCF2010ZT0R00CT-ND; OC_MOUSER 603-RC0805FR-0710KL -> (none)
- R8: value 22k -> 4,7k; OC_DIGIKEY (none) -> CR0805-FX-4701GLFTR-ND; OC_MOUSER 603-RC0805FR-0722KL -> (none)
- T2, T6: value IRF7416 -> NVR4003NT3G; device solderpi:IRF7416 -> solderpi:NVR4003NT3G; OC_DIGIKEY IRF7416TRPBFCT-ND -> NVR4003NT3GOSCT-ND
- T4: value NVR4003NT3G -> IRF7416; device solderpi:NVR4003NT3G -> solderpi:IRF7416; OC_DIGIKEY NVR4003NT3GOSCT-ND -> IRF7416TRPBFCT-ND
- X1: value NANOFIT-7 -> NEWHAVEN_OLED_256X64; device solderpi:NANOFIT-7 -> solderpi:NEWHAVEN_OLED_256X64; OC_MOUSER 538-105313-1107, 538-105307-1207 -> (none)
- X2: value PINHD-1X2 -> ULTRAFIT-290; device solderpi:PINHD-1X2 -> solderpi:ULTRAFIT-290; OC_MOUSER 855-M20-9990246 -> (none)
- X3: value NANOFIT-7 -> PINHD-1X2; device solderpi:NANOFIT-7 -> solderpi:PINHD-1X2; OC_MOUSER 538-105313-1107, 538-105307-1207 -> 855-M20-9990246
- X4: value PINHD-1X2 -> NANOFIT-7; device solderpi:PINHD-1X2 -> solderpi:NANOFIT-7; OC_MOUSER 855-M20-9990246 -> 538-105313-1107, 538-105307-1207
- X5: value NEWHAVEN_OLED_256X64 -> PINHD-1X2; device solderpi:NEWHAVEN_OLED_256X64 -> solderpi:PINHD-1X2; OC_MOUSER (none) -> 855-M20-9990246
- X6: value ULTRAFIT-290 -> NANOFIT-7; device solderpi:ULTRAFIT-290 -> solderpi:NANOFIT-7; OC_MOUSER (none) -> 538-105313-1107, 538-105307-1207
Connections:
- removed net 2_HEATER_PI: CON3.P$2
- removed net 7_GND_BL: CON3.P$1
- removed net N$1: C14.1, R8.2
- removed net N$10: IC3.VIN-, R33.2
- removed net N$11: IC3.VIN+, R31.2, R33.1
- removed net N$12: R31.1, R32.2
- removed net N$13: IC1.VIN-, R20.2
- removed net N$14: IC1.VIN+, R18.2, R20.1
- removed net N$15: X4.2
- removed net N$16: X4.1
- removed net N$17: R18.1, R19.2
- removed net N$18: X2.1
- removed net N$19: X2.2
- removed net N$2: R15.1, X3.4
- removed net N$20: R25.1, X1.4
- removed net N$21: R29.1, X1.5
- removed net N$22: R28.2, T4.G
- removed net N$23: R27.2, T5.G
- removed net N$24: R26.1, T5.D, T7.G
- removed net N$25: R21.1, T4.D, T6.G
- removed net N$26: T7.D
- removed net N$27: T6.D
- removed net N$28: IC2.VIN-, R24.2
- removed net N$29: IC2.VIN+, R22.2, R24.1
- removed net N$3: R17.1, X3.5
- removed net N$30: R22.1, R23.2
- removed net N$31: IC4.VIN-, R36.2
- removed net N$32: IC4.VIN+, R34.2, R36.1
- removed net N$33: R34.1, R35.2
- removed net N$34: X5.VDD
- removed net N$35: IC1.V+
- removed net N$36: IC3.V+
- removed net N$39: IC7.SW, L2.2
- removed net N$4: R16.2, T9.G
- removed net N$40: IC6.SW, L1.2
- removed net N$42: IC6.PG, R37.1
- removed net N$45: IC7.PG, R38.1
- removed net N$5: R2.2, T1.G
- removed net N$6: R1.1, T1.D, T2.G
- removed net N$7: R30.1, T3.G, T9.D
- removed net N$8: T2.D
- removed net N$9: T3.D
- removed net ROT0_A: C6.1, R4.1
- removed net ROT0_A_UNFIL: R3.1, R4.2, SW1G$1.A
- removed net ROT0_B: C7.1, R7.2
- removed net ROT0_B_UNFIL: R5.1, R7.1, SW1G$1.B
- removed net ROT0_SW_R: R11.1, R9.1, SW1G$2.1
- removed net ROT1_A: C9.1, R12.1
- removed net ROT1_A_UNFIL: R12.2, R6.1, SW2G$1.A
- removed net ROT1_B: C13.1, R13.2
- removed net ROT1_B_UNFIL: R10.1, R13.1, SW2G$1.B
- removed net ROT1_SW: C8.1, R11.2
- removed net ROT1_SW_R: R14.1, R8.1, SW2G$2.1
- new net 2_HEATER2_BR: CON1.P$2
- new net 3V3_PG: IC3.PG, R5.1
- new net 3V3_SW: IC3.SW, L2.2
- new net 5V_PG: IC2.PG, R4.1
- new net 5V_SW: IC2.SW, L1.2
- new net 7_GND_WH: CON1.P$1
- new net CHA0_SCL: IC1G$2.PB6, R19.1, X3.1, X4.4
- new net CHA0_SDA: IC1G$2.PB7, R21.1, X3.2, X4.5
- new net CHA0_TIP0: IC5.VIN-, R16.2, X4.1
- new net CHA0_TIP0_CUR: IC1G$1.PC1, IC5.VOUT
- new net CHA0_TIP0_PWM: IC1G$2.PA11, R8.2, T2.G
- new net CHA0_TIP0_PWM_D: R10.1, T2.D, T4.G
- new net CHA0_TIP0_SEN: IC5.VIN+, R13.2, R16.1, T4.D
- new net CHA0_TIP0_VOL: IC1G$1.PC0, R13.1, R14.2
- new net CHA0_TIP1: IC4.VIN-, R15.2, X4.2
- new net CHA0_TIP1_CUR: IC1G$1.PC3, IC4.VOUT
- new net CHA0_TIP1_PWM: IC1G$2.PA10, R7.2, T1.G
- new net CHA0_TIP1_PWM_D: R9.1, T1.D, T3.G
- new net CHA0_TIP1_SEN: IC4.VIN+, R11.2, R15.1, T3.D
- new net CHA0_TIP1_VOL: IC1G$1.PC2, R11.1, R12.2
- new net CHA1_SCL: IC1G$1.PB10, R36.1, X5.1, X6.4
- new net CHA1_SDA: IC1G$1.PB11, R38.1, X5.2, X6.5
- new net CHA1_TIP0: IC6.VIN-, R33.2, X6.1
- new net CHA1_TIP0_CUR: IC1G$1.PA1, IC6.VOUT
- new net CHA1_TIP0_PWM: IC1G$2.PA9, R25.2, T5.G
- new net CHA1_TIP0_PWM_D: R27.1, T5.D, T7.G
- new net CHA1_TIP0_SEN: IC6.VIN+, R29.2, R33.1, T7.D
- new net CHA1_TIP0_VOL: IC1G$1.PA0, R29.1, R30.2
- new net CHA1_TIP1: IC7.VIN-, R34.2, X6.2
- new net CHA1_TIP1_CUR: IC1G$1.PA3, IC7.VOUT
- new net CHA1_TIP1_PWM: IC1G$2.PA8, R26.2, T6.G
- new net CHA1_TIP1_PWM_D: R28.1, T6.D, T8.G
- new net CHA1_TIP1_SEN: IC7.VIN+, R31.2, R34.1, T8.D
- new net CHA1_TIP1_VOL: IC1G$1.PA2, R31.1, R32.2
- new net ENC0_A: C13.1, IC1G$2.PC11, R17.1
- new net ENC0_A_UNFIL: R17.2, R18.1, SW1G$1.A
- new net ENC0_B: C14.1, IC1G$2.PA15, R22.2
- new net ENC0_B_UNFIL: R20.1, R22.1, SW1G$1.B
- new net ENC0_SW: C15.1, IC1G$2.PC10, R24.2
- new net ENC0_SW_R: R23.1, R24.1, SW1G$2.1
- new net ENC1_A: C16.1, IC1G$1.PA5, R35.1
- new net ENC1_A_UNFIL: R35.2, R37.1, SW2G$1.A
- new net ENC1_B: C17.1, IC1G$1.PA7, R40.2
- new net ENC1_B_UNFIL: R39.1, R40.1, SW2G$1.B
- new net ENC1_SW: C18.1, IC1G$1.PA6, R42.2
- new net ENC1_SW_R: R41.1, R42.1, SW2G$2.1
- net +12V: now also C10.+, C8.1, C9.1, IC2.EN, IC2.VIN, IC3.EN, IC3.VIN, R10.2, R27.2, R28.2, R9.2, T4.S, T8.S, X2.1; no longer C2.1, C4.1, C5.+, IC6.EN, IC6.VIN, IC7.EN, IC7.VIN, R1.2, R21.2, R26.2, R30.2, T2.S, T6.S, X6.1
- net +3V3: now also C1.1, C12.1, C5.1, C7.1, IC1G$3.VDD@1, IC1G$3.VDD@2, IC1G$3.VDD@3, IC1G$3.VDDUSB, IC3.VOS, R18.2, R20.2, R23.2, R37.2, R39.2, R41.2, X1.VDD; no longer C15.1, C16.1, C17.1, C18.1, IC2.V+, IC4.V+, IC5G$3.VDD@1, IC5G$3.VDD@2, IC5G$3.VDD@3, IC5G$3.VDDUSB, IC7.VOS, R10.2, R14.2, R3.2, R38.2, R6.2, R9.2
- net +3V3_ANA: now also C2.1, C4.1, C6.1, IC1G$3.VDDA/VREF+, IC4.V+, IC5.V+, IC6.V+, IC7.V+, L3.1; no longer C10.1, C11.1, C12.1, IC5G$3.VDDA/VREF+
- net +5V: now also C11.1, IC2.VOS, R19.2, R21.2, R36.2, R38.2, R4.2, X4.3, X6.3; no longer C1.1, IC6.VOS, R15.2, R17.2, R25.2, R29.2, R37.2, X1.3, X3.3
- net 1_HEATER1_BR: now also CON1.P$4, CON2.P$4; no longer CON3.P$4, CON4.P$4
- net 3_+5V_GY: now also CON1.P$3, CON2.P$3; no longer CON3.P$3, CON4.P$3
- net 4_SCL_GR: now also CON1.P$6, CON2.P$6; no longer CON3.P$6, CON4.P$6
- net 5_SDA_YE: now also CON1.P$7; no longer CON3.P$7
- net 6_GND_WH: now also CON1.P$5, CON2.P$5; no longer CON3.P$5, CON4.P$5
- net AGND: now also C2.2, C4.2, C6.2, IC1G$3.VSSA/VREF-, IC4.GND, IC5.GND, IC6.GND, IC7.GND, R6.2; no longer C10.2, C11.2, C12.2, IC5G$3.VSSA/VREF-, R39.2
- net GND: now also C10.-, C11.2, C12.2, C5.2, IC1G$3.VSS@1, IC1G$3.VSS@2, IC1G$3.VSS@3, IC1G$3.VSS@4, IC2.AGND, IC2.FB, IC2.PGND, IC3.AGND, IC3.FB, IC3.PGND, R1.1, R12.1, R14.1, R25.1, R26.1, R3.1, R30.1, R6.1, R7.1, R8.1, T2.S, T6.S, X1.BS0, X1.BS1, X1.VSS@1, X1.VSS@2, X1.VSS@3, X1.VSS@4, X1.VSS@5, X1.VSS@6, X1.VSS@7, X1.VSS@8, X2.2, X4.6, X4.7, X6.6, X6.7; no longer C2.2, C4.2, C5.-, C6.2, IC1.GND, IC2.GND, IC3.GND, IC4.GND, IC5G$3.VSS@1, IC5G$3.VSS@2, IC5G$3.VSS@3, IC5G$3.VSS@4, IC6.AGND, IC6.FB, IC6.PGND, IC7.AGND, IC7.FB, IC7.PGND, R16.1, R19.1, R23.1, R27.1, R28.1, R35.1, R39.1, R41.1, T4.S, T9.S, X1.6, X1.7, X3.6, X3.7, X5.BS0, X5.BS1, X5.VSS@1, X5.VSS@2, X5.VSS@3, X5.VSS@4, X5.VSS@5, X5.VSS@6, X5.VSS@7, X5.VSS@8, X6.2
- net N$37: now also IC1G$3.PH3-BOOT0, R3.2; no longer IC5G$3.PH3-BOOT0, R41.2
- net OLED_!CS: now also IC1G$1.PB12, X1.!CS; no longer X5.!CS
- net OLED_!RESET: now also IC1G$2.PB14, R2.2, X1.!RES; no longer X5.!RES
- net OLED_D/C: now also IC1G$2.PC6, X1.D/C; no longer X5.D/C
- net OLED_SDCLK: now also IC1G$2.PB13, X1.SDCLK; no longer X5.SDCLK
- net OLED_SDIN: now also IC1G$2.PB15, X1.SDIN; no longer X5.SDIN
- net OSC_IN: now also IC1G$1.PH0-OSC_IN; no longer IC5G$1.PH0-OSC_IN
- net OSC_OUT: now also IC1G$1.PH1-OSC_OUT; no longer IC5G$1.PH1-OSC_OUT
- net RESET: now also IC1G$1.NRST, R1.2
- net SWDCLK: now also IC1G$2.PA14
- net SWDIO: now also IC1G$2.PA13
- net SWO: now also IC1G$2.PB3
