File: pcb/iron.brd (EAGLE design)
At the start: 8 x 24 mm, 22 parts, among them IC1 AT24CS04-SOT23, IC2 TS507CLT, IC3 AD7995, IC4 ESDA6V1SC5, X1 LUMBERG_KLB_4

Commit message: reworked iron parts
Parts:
- R1: value 20k 0,1% -> 1k
- R2: value 68k @25°C, 1%, ß=3985 K -> 1k @25°C, 1%, ß=3650 K
- R4: value 5,1M -> 4M7
- R6: value 1k -> 100k
Changed lines of the file:
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@@
 <elements>
 <element name="X1" library="solderpi" library_urn="urn:adsk.eagle:library:1437534" package="3.5_MM_AUDIO_JACK" package3d_urn="urn:adsk.eagle:package:1437574/2" value="LUMBERG_KLB_4" x="4" y="23.4" smashed="yes" rot="MR0"/>
-<element name="R1" library="common" library_urn="urn:adsk.eagle:library:8241912" package="R0603" package3d_urn="urn:adsk.eagle:package:8241925/3" value="20k 0,1%" x="5.6" y="15.85" smashed="yes" rot="MR180">
+<element name="R1" library="common" library_urn="urn:adsk.eagle:library:8241912" package="R0603" package3d_urn="urn:adsk.eagle:package:8241925/3" value="1k" x="5.6" y="15.85" smashed="yes" rot="MR180">
 <attribute name="NAME" x="7.0754" y="15.85" size="0.8128" layer="26" rot="MR90" align="bottom-center"/>
-<attribute name="OC_DIGIKEY" value="P20KDBCT-ND" x="5.6" y="15.85" size="1.778" layer="28" rot="MR180" display="off"/>
+<attribute name="OC_DIGIKEY" value="P1.0KDBCT-ND" x="5.6" y="15.85" size="1.778" layer="28" rot="MR180" display="off"/>
 <attribute name="VALUE" x="4.965" y="18.39" size="1.27" layer="28" rot="MR180"/>
 </element>
-<element name="R2" library="common" library_urn="urn:adsk.eagle:library:8241912" package="R0603" package3d_urn="urn:adsk.eagle:package:8241925/3" value="68k @25°C, 1%, ß=3985 K" x="2.4" y="15.85" smashed="yes" rot="MR180">
+<element name="R2" library="common" library_urn="urn:adsk.eagle:library:8241912" package="R0603" package3d_urn="urn:adsk.eagle:package:8241925/3" value="1k @25°C, 1%, ß=3650 K" x="2.4" y="15.85" smashed="yes" rot="MR180">
 <attribute name="NAME" x="0.9246" y="15.85" size="0.8128" layer="26" rot="MR90" align="top-center"/>
-<attribute name="OC_DIGIKEY" value="BC2555CT-ND" x="2.4" y="15.85" size="1.778" layer="28" rot="MR180" display="off"/>
+<attribute name="OC_DIGIKEY" value="P123687CT-ND" x="2.4" y="15.85" size="1.778" layer="28" rot="MR180" display="off"/>
 <attribute name="VALUE" x="1.765" y="18.39" size="1.27" layer="28" rot="MR180"/>
 </element>
@@
 <attribute name="NAME" x="2.15" y="8.7032" size="0.8128" layer="21" align="bottom-center"/>
 </element>
-<element name="R4" library="common" library_urn="urn:adsk.eagle:library:8241912" package="R0603" package3d_urn="urn:adsk.eagle:package:8241925/3" value="5,1M" x="5.45" y="6.25" smashed="yes" rot="R180">
+<element name="R4" library="common" library_urn="urn:adsk.eagle:library:8241912" package="R0603" package3d_urn="urn:adsk.eagle:package:8241925/3" value="4M7" x="5.45" y="6.25" smashed="yes" rot="R180">
 <attribute name="NAME" x="7.0754" y="6.25" size="0.8128" layer="25" rot="R90" align="top-center"/>
-<attribute name="OC_MOUSER" value="71-CRCW08055M10FKEA" x="5.45" y="6.25" size="1.778" layer="27" rot="R180" display="off"/>
+<attribute name="OC_DIGIKEY" value="311-4.70MHRCT-ND" x="5.45" y="6.25" size="1.778" layer="27" rot="R180" display="off"/>
 <attribute name="VALUE" x="6.085" y="8.79" size="1.27" layer="27" rot="R180"/>
 </element>
@@
 <attribute name="VALUE" x="4.815" y="5.11" size="1.27" layer="27"/>
 </element>
-<element name="R6" library="common" library_urn="urn:adsk.eagle:library:8241912" package="R0603" package3d_urn="urn:adsk.eagle:package:8241925/3" value="1k" x="5.45" y="9.05" smashed="yes" rot="R180">
+<element name="R6" library="common" library_urn="urn:adsk.eagle:library:8241912" package="R0603" package3d_urn="urn:adsk.eagle:package:8241925/3" value="100k" x="5.45" y="9.05" smashed="yes" rot="R180">
 <attribute name="NAME" x="7.0754" y="9.05" size="0.8128" layer="25" rot="R90" align="top-center"/>
-<attribute name="OC_DIGIKEY" value=" RMCF0603FT1K00CT-ND" x="5.45" y="9.05" size="1.778" layer="27" rot="R180" display="off"/>
+<attribute name="OC_DIGIKEY" value="RMCF0603FT100KCT-ND" x="5.45" y="9.05" size="1.778" layer="27" rot="R180" display="off"/>
 <attribute name="VALUE" x="6.085" y="11.59" size="1.27" layer="27" rot="R180"/>
 </element>
 <element name="C1" library="common" library_urn="urn:adsk.eagle:library:8241912" package="C0603" package3d_urn="urn:adsk.eagle:package:8241929/3" value="100pF" x="5.45" y="4.9" smashed="yes">
 <attribute name="NAME" x="7.0024" y="4.9" size="0.8128" layer="25" rot="R90" align="top-center"/>
-<attribute name="OC_MOUSER" value="710-885012207080" x="5.45" y="4.9" size="1.778" layer="27" display="off"/>
+<attribute name="OC_DIGIKEY" value="478-7926-1-ND" x="5.45" y="4.9" size="1.778" layer="27" display="off"/>
 <attribute name="VALUE" x="4.18" y="2.36" size="1.27" layer="27"/>
 </element>
 <element name="C2" library="common" library_urn="urn:adsk.eagle:library:8241912" package="C0603" package3d_urn="urn:adsk.eagle:package:8241929/3" value="10nF" x="4" y="15.9" smashed="yes" rot="R270">
 <attribute name="NAME" x="4" y="17.3254" size="0.8128" layer="25" rot="R90" align="center-left"/>
-<attribute name="OC_MOUSER" value="710-885012207092 " x="4" y="15.9" size="1.778" layer="27" rot="R270" display="off"/>
+<attribute name="OC_DIGIKEY" value="478-6209-1-ND" x="4" y="15.9" size="1.778" layer="27" rot="R270" display="off"/>
 <attribute name="VALUE" x="1.46" y="17.17" size="1.27" layer="27" rot="R270"/>
 </element>

Commit message: shottky diode added to iron/tweezer
Parts:
- added C3, C4: 1µF, common:C0603
- added D1: BAT54H, solderpi:SOD123-F
- moved R1 2.00 mm to (5.60, 17.9)
- moved R2 2.00 mm to (2.40, 17.9)
- moved R7 2.00 mm to (2.65, 17.9)
- moved C1 2.00 mm to (5.45, 6.90)
- moved GND 2.00 mm to (6.30, 20.5)
- moved IC1 2.00 mm to (4.00, 10.7)
- moved IC2 2.00 mm to (4.00, 14.0)
- moved IC3 2.00 mm to (4.00, 14.5)
- moved IC4 2.00 mm to (4.00, 6.80)
- moved PWR 2.00 mm to (1.70, 20.5)
- moved R10 2.00 mm to (1.55, 13.4)
- moved R3 2.00 mm to (2.15, 8.25)
- moved R4 2.00 mm to (5.45, 8.25)
- moved R5 2.00 mm to (5.45, 9.65)
- moved R6 2.00 mm to (5.45, 11.1)
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Connections:
- new net N$1: C1.1, C4.1, D1.1, R4.2
- net +5V: now also C3.1, D1.2; no longer C1.1, R4.2
- net GND: now also C3.2, C4.2
Routing:
- net GND: track 42.6 -> 53.4 mm
- net N$1: track 0.00 -> 5.10 mm
- net SDA: track 15.5 -> 17.5 mm
- net SCL: track 13.4 -> 15.4 mm
Other:
- board size 8 x 24 mm -> 8 x 26 mm

Commit message: boms reworked
Parts:
- moved D1 0.50 mm to (5.30, 4.40)
- moved C1 0.50 mm to (5.45, 7.40)
- moved C2 0.50 mm to (4.00, 18.4)
- moved C3 0.50 mm to (5.40, 4.30)
- moved C4 0.50 mm to (5.45, 6.10)
- moved GND 0.50 mm to (6.30, 21.0)
- moved IC1 0.50 mm to (4.00, 11.2)
- moved IC2 0.50 mm to (4.00, 14.5)
- moved IC3 0.50 mm to (4.00, 15.0)
- moved IC4 0.50 mm to (4.00, 7.30)
- moved PWR 0.50 mm to (1.70, 21.0)
- moved R1 0.50 mm to (5.60, 18.4)
- moved R10 0.50 mm to (1.55, 13.9)
- moved R2 0.50 mm to (2.40, 18.4)
- moved R3 0.50 mm to (2.15, 8.75)
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Routing:
- net +5V: track 37.1 -> 38.1 mm
- net SDA: track 17.5 -> 18.0 mm
- net SCL: track 15.4 -> 15.9 mm
Other:
- board size 8 x 26 mm -> 8 x 26.5 mm
