File: kicad/rotary_enc.sch (KiCad schematic (older format))
At the start: 20 parts, among them SW401 ROT_ENC_SWITCH, SW402 ROT_ENC_SWITCH

Commit message: refactored debug connector
Parts:
- SW401, SW402: Voelkner (none) -> D77476
Changed lines of the file:
@@
 F 2 "solder_station:EC12E" H 2350 3625 50  0001 C CNN
 F 3 "" H 2350 3625 50  0001 C CNN
+F 4 "D77476" H 2450 3550 50  0001 C CNN "Voelkner"
 	1    2450 3550
 	1    0    0    -1
@@
 F 2 "solder_station:EC12E" H 6550 3625 50  0001 C CNN
 F 3 "" H 6550 3625 50  0001 C CNN
+F 4 "D77476" H 6650 3550 50  0001 C CNN "Voelkner"
 	1    6650 3550
 	1    0    0    -1
